Commit message: got it to have gazebo again

File: urdf/sentry.urdf.xacro (robot description, xacro)
@@ -73,8 +73,7 @@
     <xacro:box_inertia m="0.5" w="${head_width}" h="${head_height}" d="${head_length}" />
   </link>
-  <!-- 4. Sensors (Fixed to Head) -->
   <joint name="lidar_joint" type="fixed">
     <parent link="head_link" />
-    <child link="lidar_link" />
+    <child link="lidar" />
     <!-- Placed on the front edge of the head -->
     <origin xyz="0.12218 -0.17882 0" rpy="0 0 ${pi/2}" />

Commit message: added software lidar to urdf

File: urdf/sentry.urdf.xacro (robot description, xacro)
@@ -19,8 +19,4 @@
   <!-- 1. Robot Footprint (The Ground Reference) -->
   <link name="base_footprint">
-    <inertial>
-      <mass value="0.0001" />
-      <inertia ixx="0.0001" ixy="0" ixz="0" iyy="0.0001" iyz="0" izz="0.0001" />
-    </inertial>
   </link>
   <joint name="base_joint" type="fixed">
@@ -76,5 +72,4 @@
     <parent link="head_link" />
     <child link="lidar" />
-    <!-- Placed on the front edge of the head -->
     <origin xyz="0.12218 -0.17882 0" rpy="0 0 ${pi/2}" />
   </joint>
@@ -97,32 +92,31 @@
       <inertia ixx="0.001" ixy="0" ixz="0" iyy="0.001" iyz="0" izz="0.001" />
     </inertial>
+    <sensor name="lidar" type="gpu_lidar">
+      <always_on>true</always_on>
+      <visualize>true</visualize>
+      <update_rate>5</update_rate>
+      <topic>scan</topic>
+      <gz_frame_id>lidar</gz_frame_id>
+      <lidar>
+        <scan>
+          <horizontal>
+            <samples>360</samples>
+            <resolution>1.000000</resolution>
+            <min_angle>0.000000</min_angle>
+            <max_angle>6.280000</max_angle>
+          </horizontal>
+        </scan>
+        <range>
+          <min>0.120000</min>
+          <max>3.5</max>
+          <resolution>0.015000</resolution>
+        </range>
+        <noise>
+          <type>gaussian</type>
+          <mean>0.0</mean>
+          <stddev>0.01</stddev>
+        </noise>
+      </lidar>
+    </sensor>
   </link>
-  <!-- <gazebo reference="laser"> -->
-  <!-- <sensor name="lidar" type="ray"> -->
-  <!-- <pose>0 0 0 0 0 0</pose> -->
-  <!-- <visualize>true</visualize> -->
-  <!-- <update_rate>10</update_rate> -->
-  <!-- <ray> -->
-  <!-- <scan> -->
-  <!-- <horizontal> -->
-  <!-- <samples>360</samples> -->
-  <!-- <resolution>1</resolution> -->
-  <!-- <min_angle>-3.14</min_angle> -->
-  <!-- <max_angle>3.14</max_angle> -->
-  <!-- </horizontal> -->
-  <!-- </scan> -->
-  <!-- <range> -->
-  <!-- <min>0.3</min> -->
-  <!-- <max>12.0</max> -->
-  <!-- </range> -->
-  <!-- </ray> -->
-  <!-- <plugin name="gazebo_ros_ray_sensor" filename="libgazebo_ros_ray_sensor.so"> -->
-  <!-- <ros> -->
-  <!-- <remapping>~/out:=scan</remapping> -->
-  <!-- </ros> -->
-  <!-- <output_type>sensor_msgs/LaserScan</output_type> -->
-  <!-- <frame_name>laser</frame_name> -->
-  <!-- </plugin> -->
-  <!-- </sensor> -->
-  <!-- </gazebo> -->
 </robot>

Commit message: added new world

File: urdf/sentry.urdf.xacro (robot description, xacro)
@@ -92,4 +92,7 @@
       <inertia ixx="0.001" ixy="0" ixz="0" iyy="0.001" iyz="0" izz="0.001" />
     </inertial>
+  </link>
+  <gazebo reference="lidar">
+    <gz_frame_id>lidar</gz_frame_id>
     <sensor name="lidar" type="gpu_lidar">
       <always_on>true</always_on>
@@ -119,4 +122,4 @@
       </lidar>
     </sensor>
-  </link>
+  </gazebo>
 </robot>

Commit message: removed 1000 screws

File: urdf/sentry.urdf.xacro (robot description, xacro)
@@ -1,125 +1,70 @@
-<?xml version="1.0"?>
-<robot name="sentry" xmlns:xacro="http://ros.org">
-  <!-- Define robot constants -->
-  <xacro:property name="base_radius" value="0.2975" />
-  <xacro:property name="base_height" value="0.220" />
-  <xacro:property name="head_length" value="0.29528" />
-  <xacro:property name="head_width" value="0.1524" />
-  <xacro:property name="head_height" value="0.18398" />
-  <!-- Inertial Macros -->
-  <xacro:macro name="box_inertia" params="m w h d">
-    <inertial>
-      <origin xyz="0 0 0" rpy="0 0 0" />
-      <mass value="${m}" />
-      <inertia ixx="${(m/12) * (h*h + d*d)}" ixy="0.0" ixz="0.0"
-        iyy="${(m/12) * (w*w + d*d)}" iyz="0.0"
-        izz="${(m/12) * (w*w + h*h)}" />
-    </inertial>
-  </xacro:macro>
-  <!-- 1. Robot Footprint (The Ground Reference) -->
-  <link name="base_footprint">
-  </link>
-  <joint name="base_joint" type="fixed">
-    <parent link="base_footprint" />
-    <child link="base_link" />
-    <origin xyz="0 0 ${base_height/2}" rpy="0 0 0" />
-  </joint>
-  <!-- 2. Robot Base (The Cylinder) -->
-  <link name="base_link">
-    <visual>
-      <geometry>
-        <cylinder radius="${base_radius}" length="${base_height}" />
-      </geometry>
-      <material name="Dark_Cyan">
-        <color rgba="0 0.8 0.8 0.8" />
-      </material>
-    </visual>
-    <collision>
-      <geometry>
-        <cylinder radius="${base_radius}" length="${base_height}" />
-      </geometry>
-    </collision>
-    <inertial>
-      <mass value="5.0" />
-      <inertia ixx="0.1" ixy="0" ixz="0" iyy="0.1" iyz="0" izz="0.2" />
-    </inertial>
-  </link>
-  <!-- 3. Robot Head (The Rotating Box) -->
-  <joint name="head_joint" type="continuous">
-    <parent link="base_link" />
-    <child link="head_link" />
-    <!-- Centers the head slightly above the top of the base cylinder -->
-    <origin xyz="0 0 ${base_height/2 + 0.05}" rpy="0 0 0" />
-    <axis xyz="0 0 1" />
-  </joint>
-  <link name="head_link">
-    <visual>
-      <geometry>
-        <box size="${head_length} ${head_width} ${head_height}" />
-      </geometry>
-      <material name="Cyan">
-        <color rgba="0 1.0 1.0 1.0" />
-      </material>
-    </visual>
-    <collision>
-      <geometry>
-        <box size="${head_length} ${head_width} ${head_height}" />
-      </geometry>
-    </collision>
-    <xacro:box_inertia m="0.5" w="${head_width}" h="${head_height}" d="${head_length}" />
-  </link>
-  <joint name="lidar_joint" type="fixed">
-    <parent link="head_link" />
-    <child link="lidar" />
-    <origin xyz="0.12218 -0.17882 0" rpy="0 0 ${pi/2}" />
-  </joint>
-  <link name="lidar">
-    <visual>
-      <geometry>
-        <cylinder radius="0.05" length="0.04" />
-      </geometry>
-      <material name="black">
-        <color rgba="0 0 0 1" />
-      </material>
-    </visual>
-    <collision>
-      <geometry>
-        <cylinder radius="0.05" length="0.04" />
-      </geometry>
-    </collision>
-    <inertial>
-      <mass value="0.1" />
-      <inertia ixx="0.001" ixy="0" ixz="0" iyy="0.001" iyz="0" izz="0.001" />
-    </inertial>
-  </link>
-  <gazebo reference="lidar">
-    <gz_frame_id>lidar</gz_frame_id>
-    <sensor name="lidar" type="gpu_lidar">
-      <always_on>true</always_on>
-      <visualize>true</visualize>
-      <update_rate>5</update_rate>
-      <topic>scan</topic>
-      <gz_frame_id>lidar</gz_frame_id>
-      <lidar>
-        <scan>
-          <horizontal>
-            <samples>360</samples>
-            <resolution>1.000000</resolution>
-            <min_angle>0.000000</min_angle>
-            <max_angle>6.280000</max_angle>
-          </horizontal>
-        </scan>
-        <range>
-          <min>0.120000</min>
-          <max>3.5</max>
-          <resolution>0.015000</resolution>
-        </range>
-        <noise>
-          <type>gaussian</type>
-          <mean>0.0</mean>
-          <stddev>0.01</stddev>
-        </noise>
-      </lidar>
-    </sensor>
-  </gazebo>
+<!--URDF generated by ONSHAPE BY PTC INC, 1.217-->
+<robot name="assembly_3">
+    <link name="part_1">
+        <inertial>
+            <mass value="0.0701287" />
+            <origin xyz="1.20374e-17 2.46519e-32 0.126108" rpy="0 -0 0" />
+            <inertia ixx="0.00192346" ixy="0" ixz="0" iyy="0.00192346" iyz="0" izz="0.00310341" />
+        </inertial>
+        <visual>
+            <origin xyz="0 -1.82166e-17 0.0734155" rpy="0 -0 0" />
+            <geometry>
+                <mesh filename="package://assembly_3/meshes/Part_1.stl" scale="1 1 1" />
+            </geometry>
+            <material name="0.615686_0.811765_0.929412_0.000000_0.000000">
+                <color rgba="0.615686 0.811765 0.929412 1" />
+            </material>
+        </visual>
+    </link>
+    <link name="part_1_1">
+        <inertial>
+            <mass value="0.00421105" />
+            <origin xyz="0.00100261 -0.00244355 0.0730117" rpy="0 -0 2.48157" />
+            <inertia ixx="1.8557e-05" ixy="4.2327e-06" ixz="1.56708e-08" iyy="1.90292e-05" iyz="-3.81928e-08" izz="2.21682e-05" />
+        </inertial>
+        <visual>
+            <origin xyz="-1.68946e-18 -2.17675e-18 0" rpy="0 -0 2.48157" />
+            <geometry>
+                <mesh filename="package://assembly_3/meshes/Part_1_1.stl" scale="1 1 1" />
+            </geometry>
+            <material name="0.615686_0.811765_0.929412_0.000000_0.000000">
+                <color rgba="0.615686 0.811765 0.929412 1" />
+            </material>
+        </visual>
+    </link>
+    <link name="part_1_2">
+        <inertial>
+            <mass value="0.00018588" />
+            <origin xyz="-6.05411e-19 -4.2157e-19 0.02065" rpy="0 -0 0.608263" />
+            <inertia ixx="9.29949e-08" ixy="0" ixz="0" iyy="9.29949e-08" iyz="0" izz="1.33148e-07" />
+        </inertial>
+        <visual>
+            <origin xyz="1.3244e-18 -1.90196e-18 0" rpy="0 -0 0.608263" />
+            <geometry>
+                <mesh filename="package://assembly_3/meshes/Part_1_2.stl" scale="1 1 1" />
+            </geometry>
+            <material name="0.615686_0.811765_0.929412_0.000000_0.000000">
+                <color rgba="0.615686 0.811765 0.929412 1" />
+            </material>
+        </visual>
+    </link>
+    <link name="root" />
+    <joint name="fastened_1" type="fixed">
+        <origin xyz="0 1.38778e-17 -8.69386e-19" rpy="-1.5708 -0 3.14159" />
+        <axis xyz="0 0 -1" />
+        <parent link="root" />
+        <child link="part_1" />
+    </joint>
+    <joint name="headlink" type="continuous">
+        <origin xyz="3.00043e-17 -1.82344e-18 0.252215" rpy="0 -0 -3.14159" />
+        <axis xyz="0 0 -1" />
+        <parent link="part_1" />
+        <child link="part_1_1" />
+    </joint>
+    <joint name="lidar" type="continuous">
+        <origin xyz="0.0884778 -0.20163 0.0718" rpy="0 0 -0.660022" />
+        <axis xyz="0 0 -1" />
+        <parent link="part_1_1" />
+        <child link="part_1_2" />
+    </joint>
 </robot>
