Commit message: removed 1000 screws

File: urdf/sentry.urdf.xacro (robot description, xacro)
@@ -1,1548 +1,14 @@
-<!--URDF generated by ONSHAPE BY PTC INC, 1.216-->
-<robot name="sentry" xmlns:xacro="http://ros.org">
-    <xacro:property name="pkg_path" value="package://sentry_pkg" />
-    <link name="base_footprint"/>
-    <link name="base_link"/>
-    <joint name="base_footprint_to_base_link" type="fixed">
-        <parent link="base_footprint"/>
-        <child link="base_link"/>
-        <origin xyz="0 0 0.05" rpy="0 0 0"/>
-    </joint>
-    <joint name="base_link_to_onshape_root" type="fixed">
-        <parent link="base_link"/>
-        <child link="root"/>
-        <origin xyz="0 0 0" rpy="0 0 0"/>
-    </joint>
-    <link name="000">
+<!--URDF generated by ONSHAPE BY PTC INC, 1.217-->
+<robot name="assembly_3">
+    <link name="part_1">
         <inertial>
-            <mass value="1.63637e-07" />
-            <origin xyz="1.69387e-12 0.0047 0.0254268" rpy="0 -0 0" />
-            <inertia ixx="1.34286e-12" ixy="0" ixz="0" iyy="1.34286e-12" iyz="0" izz="8.22314e-13" />
+            <mass value="0.0701287" />
+            <origin xyz="1.20374e-17 2.46519e-32 0.126108" rpy="0 -0 0" />
+            <inertia ixx="0.00192346" ixy="0" ixz="0" iyy="0.00192346" iyz="0" izz="0.00310341" />
         </inertial>
         <visual>
-            <origin xyz="0 0 0" rpy="0 -0 0" />
+            <origin xyz="0 -1.82166e-17 0.0734155" rpy="0 -0 0" />
             <geometry>
-                <mesh filename="package://sentry_pkg/meshes/_000.stl" scale="1 1 1" />
-            </geometry>
-            <material name="0.196078_0.196078_0.196078_0.000000_0.000000">
-                <color rgba="0.196078 0.196078 0.196078 1" />
-            </material>
-        </visual>
-    </link>
-    <link name="000_1">
-        <inertial>
-            <mass value="2.87618e-05" />
-            <origin xyz="0.000206207 0.00944711 -0.00214079" rpy="0 -0 0" />
-            <inertia ixx="8.48719e-09" ixy="1.03855e-11" ixz="-1.31637e-11" iyy="2.01238e-08" iyz="-5.68809e-11" izz="1.1955e-08" />
-        </inertial>
-        <visual>
-            <origin xyz="0 0 0" rpy="0 -0 0" />
-            <geometry>
-                <mesh filename="package://sentry_pkg/meshes/_000_1.stl" scale="1 1 1" />
-            </geometry>
-            <material name="0.400000_0.400000_0.400000_0.000000_0.000000">
-                <color rgba="0.4 0.4 0.4 1" />
-            </material>
-        </visual>
-    </link>
-    <link name="000_2">
-        <inertial>
-            <mass value="4.84713e-06" />
-            <origin xyz="-0.000243953 0.00570155 -0.00444345" rpy="0 -0 0" />
-            <inertia ixx="9.76479e-10" ixy="9.78988e-12" ixz="5.85577e-11" iyy="2.06522e-09" iyz="1.79663e-11" izz="1.11938e-09" />
-        </inertial>
-        <visual>
-            <origin xyz="0 0 0" rpy="0 -0 0" />
-            <geometry>
-                <mesh filename="package://sentry_pkg/meshes/_000_2.stl" scale="1 1 1" />
-            </geometry>
-            <material name="0.196078_0.196078_0.196078_0.000000_0.000000">
-                <color rgba="0.196078 0.196078 0.196078 1" />
-            </material>
-        </visual>
-    </link>
-    <link name="000_3">
-        <inertial>
-            <mass value="8.61711e-06" />
-            <origin xyz="0.0220919 0.00162236 -0.0312108" rpy="0 -0 0" />
-            <inertia ixx="3.37959e-09" ixy="7.70106e-14" ixz="5.11165e-12" iyy="8.51082e-09" iyz="-1.1979e-11" izz="5.17026e-09" />
-        </inertial>
-        <visual>
-            <origin xyz="0.022 0 -0.0287" rpy="0 -0 0" />
-            <geometry>
-                <mesh filename="package://sentry_pkg/meshes/_000_3.stl" scale="1 1 1" />
-            </geometry>
-            <material name="0.400000_0.400000_0.400000_0.000000_0.000000">
-                <color rgba="0.4 0.4 0.4 1" />
-            </material>
-        </visual>
-    </link>
-    <link name="000_4">
-        <inertial>
-            <mass value="9.64332e-07" />
-            <origin xyz="-8.35252e-05 0.0131856 -0.017571" rpy="0 -0 0" />
-            <inertia ixx="2.5523e-11" ixy="-9.95213e-14" ixz="5.0269e-13" iyy="1.10533e-10" iyz="3.4526e-14" izz="8.57133e-11" />
-        </inertial>
-        <visual>
-            <origin xyz="0 0 0" rpy="0 -0 0" />
-            <geometry>
-                <mesh filename="package://sentry_pkg/meshes/_000_4.stl" scale="1 1 1" />
-            </geometry>
-            <material name="0.901961_0.901961_0.901961_0.000000_0.000000">
-                <color rgba="0.901961 0.901961 0.901961 1" />
-            </material>
-        </visual>
-    </link>
-    <link name="000_5">
-        <inertial>
-            <mass value="1.27235e-08" />
-            <origin xyz="-0.0269 0.000725 -0.0275" rpy="0 -0 0" />
-            <inertia ixx="1.19627e-14" ixy="0" ixz="0" iyy="2.0612e-14" iyz="0" izz="1.19627e-14" />
-        </inertial>
-        <visual>
-            <origin xyz="0 0 0" rpy="0 -0 0" />
-            <geometry>
-                <mesh filename="package://sentry_pkg/meshes/_000_5.stl" scale="1 1 1" />
-            </geometry>
-            <material name="0.250980_0.250980_0.250980_0.000000_0.000000">
-                <color rgba="0.25098 0.25098 0.25098 1" />
-            </material>
-        </visual>
-    </link>
-    <link name="000_6">
-        <inertial>
-            <mass value="3.78562e-08" />
-            <origin xyz="0.0269 0.00379554 0.021" rpy="0 -0 0" />
-            <inertia ixx="3.32976e-13" ixy="0" ixz="0" iyy="3.31784e-14" iyz="0" izz="3.32976e-13" />
-        </inertial>
-        <visual>
-            <origin xyz="0 0 0" rpy="0 -0 0" />
-            <geometry>
-                <mesh filename="package://sentry_pkg/meshes/_000_6.stl" scale="1 1 1" />
-            </geometry>
-            <material name="0.250980_0.250980_0.250980_0.000000_0.000000">
-                <color rgba="0.25098 0.25098 0.25098 1" />
-            </material>
-        </visual>
-    </link>
-    <link name="000_7">
-        <inertial>
-            <mass value="1.72285e-06" />
-            <origin xyz="5.0161e-07 0.00975486 0.0114898" rpy="0 -0 0" />
-            <inertia ixx="5.98453e-11" ixy="-4.81504e-15" ixz="0" iyy="3.00362e-10" iyz="7.54289e-13" izz="2.6455e-10" />
-        </inertial>
-        <visual>
-            <origin xyz="0 0 0" rpy="0 -0 0" />
-            <geometry>
-                <mesh filename="package://sentry_pkg/meshes/_000_7.stl" scale="1 1 1" />
-            </geometry>
-            <material name="0.196078_0.196078_0.196078_0.000000_0.000000">
-                <color rgba="0.196078 0.196078 0.196078 1" />
-            </material>
-        </visual>
-    </link>
-    <link name="000_8">
-        <inertial>
-            <mass value="1.27235e-08" />
-            <origin xyz="-0.0269 0.000725 0.021" rpy="0 -0 0" />
-            <inertia ixx="1.19627e-14" ixy="0" ixz="0" iyy="2.0612e-14" iyz="0" izz="1.19627e-14" />
-        </inertial>
-        <visual>
-            <origin xyz="0 0 0" rpy="0 -0 0" />
-            <geometry>
-                <mesh filename="package://sentry_pkg/meshes/_000_8.stl" scale="1 1 1" />
-            </geometry>
-            <material name="0.250980_0.250980_0.250980_0.000000_0.000000">
-                <color rgba="0.25098 0.25098 0.25098 1" />
-            </material>
-        </visual>
-    </link>
-    <link name="lidar">
-        <inertial>
-            <mass value="3.78562e-08" />
-            <origin xyz="0.0269 0.00379554 -0.0275" rpy="0 -0 0" />
-            <inertia ixx="3.32976e-13" ixy="0" ixz="0" iyy="3.31784e-14" iyz="0" izz="3.32976e-13" />
-        </inertial>
-        <visual>
-            <origin xyz="0 0 0" rpy="0 -0 0" />
-            <geometry>
-                <mesh filename="package://sentry_pkg/meshes/_000_9.stl" scale="1 1 1" />
-            </geometry>
-            <material name="0.250980_0.250980_0.250980_0.000000_0.000000">
-                <color rgba="0.25098 0.25098 0.25098 1" />
-            </material>
-        </visual>
-    </link>
-    <link name="1">
-        <inertial>
-            <mass value="9.41379e-07" />
-            <origin xyz="0.00160638 0.0055 -0.00398923" rpy="0 -0 0" />
-            <inertia ixx="1.775e-11" ixy="0" ixz="2.82208e-13" iyy="3.57375e-11" iyz="0" izz="3.66023e-11" />
-        </inertial>
-        <visual>
-            <origin xyz="0 0 0" rpy="0 -0 0" />
-            <geometry>
-                <mesh filename="package://sentry_pkg/meshes/_1.stl" scale="1 1 1" />
-            </geometry>
-            <material name="0.666667_0.698039_0.764706_0.000000_0.000000">
-                <color rgba="0.666667 0.698039 0.764706 1" />
-            </material>
-        </visual>
-    </link>
-    <link name="1111">
-        <inertial>
-            <mass value="0.00117942" />
-            <origin xyz="-0.00960332 0.000184097 0.000182757" rpy="0 -0 0" />
-            <inertia ixx="5.73556e-07" ixy="-1.48664e-09" ixz="5.72675e-09" iyy="1.51998e-06" iyz="1.56233e-10" izz="9.4865e-07" />
-        </inertial>
-        <visual>
-            <origin xyz="0.0345519 0.00182103 0.0272507" rpy="0 -0 0" />
-            <geometry>
-                <mesh filename="package://sentry_pkg/meshes/_1111.stl" scale="1 1 1" />
-            </geometry>
-            <material name="0.910000_0.910000_0.910000_0.000000_0.000000">
-                <color rgba="0.91 0.91 0.91 1" />
-            </material>
-        </visual>
-        <visual>
-            <origin xyz="0.0345519 0.00182103 0.0272507" rpy="0 -0 0" />
-            <geometry>
-                <mesh filename="package://sentry_pkg/meshes/_1111_1.stl" scale="1 1 1" />
-            </geometry>
-            <material name="0.910000_0.910000_0.910000_0.000000_0.000000">
-                <texture />
-                <color rgba="0.91 0.91 0.91 1" />
-            </material>
-        </visual>
-        <visual>
-            <origin xyz="0.0345519 0.00182103 0.0272507" rpy="0 -0 0" />
-            <geometry>
-                <mesh filename="package://sentry_pkg/meshes/_1111_2.stl" scale="1 1 1" />
-            </geometry>
-            <material name="0.910000_0.910000_0.910000_0.000000_0.000000">
-                <texture />
-                <color rgba="0.91 0.91 0.91 1" />
-            </material>
-        </visual>
-        <visual>
-            <origin xyz="0.0345519 0.00182103 0.0272507" rpy="0 -0 0" />
-            <geometry>
-                <mesh filename="package://sentry_pkg/meshes/_1111_3.stl" scale="1 1 1" />
-            </geometry>
-            <material name="0.910000_0.910000_0.910000_0.000000_0.000000">
-                <texture />
-                <color rgba="0.91 0.91 0.91 1" />
-            </material>
-        </visual>
-        <visual>
-            <origin xyz="0.0345519 0.00182103 0.0272507" rpy="0 -0 0" />
-            <geometry>
-                <mesh filename="package://sentry_pkg/meshes/_1111_4.stl" scale="1 1 1" />
-            </geometry>
-            <material name="0.910000_0.910000_0.910000_0.000000_0.000000">
-                <texture />
-                <color rgba="0.91 0.91 0.91 1" />
-            </material>
-        </visual>
-        <visual>
-            <origin xyz="0.0345519 0.00182103 0.0272507" rpy="0 -0 0" />
-            <geometry>
-                <mesh filename="package://sentry_pkg/meshes/_1111_5.stl" scale="1 1 1" />
-            </geometry>
-            <material name="0.910000_0.910000_0.910000_0.000000_0.000000">
-                <texture />
-                <color rgba="0.91 0.91 0.91 1" />
-            </material>
-        </visual>
-        <visual>
-            <origin xyz="0.0345519 0.00182103 0.0272507" rpy="0 -0 0" />
-            <geometry>
-                <mesh filename="package://sentry_pkg/meshes/_1111_6.stl" scale="1 1 1" />
-            </geometry>
-            <material name="0.910000_0.910000_0.910000_0.000000_0.000000">
-                <texture />
-                <color rgba="0.91 0.91 0.91 1" />
-            </material>
-        </visual>
-        <visual>
-            <origin xyz="0.0345519 0.00182103 0.0272507" rpy="0 -0 0" />
-            <geometry>
-                <mesh filename="package://sentry_pkg/meshes/_1111_7.stl" scale="1 1 1" />
-            </geometry>
-            <material name="0.910000_0.910000_0.910000_0.000000_0.000000">
-                <texture />
-                <color rgba="0.91 0.91 0.91 1" />
-            </material>
-        </visual>
-        <visual>
-            <origin xyz="0.0345519 0.00182103 0.0272507" rpy="0 -0 0" />
-            <geometry>
-                <mesh filename="package://sentry_pkg/meshes/_1111_8.stl" scale="1 1 1" />
-            </geometry>
-            <material name="0.910000_0.910000_0.910000_0.000000_0.000000">
-                <texture />
-                <color rgba="0.91 0.91 0.91 1" />
-            </material>
-        </visual>
-        <visual>
-            <origin xyz="0.0345519 0.00182103 0.0272507" rpy="0 -0 0" />
-            <geometry>
-                <mesh filename="package://sentry_pkg/meshes/_1111_9.stl" scale="1 1 1" />
-            </geometry>
-            <material name="0.910000_0.910000_0.910000_0.000000_0.000000">
-                <texture />
-                <color rgba="0.91 0.91 0.91 1" />
-            </material>
-        </visual>
-        <visual>
-            <origin xyz="0.0345519 0.00182103 0.0272507" rpy="0 -0 0" />
-            <geometry>
-                <mesh filename="package://sentry_pkg/meshes/_1111_10.stl" scale="1 1 1" />
-            </geometry>
-            <material name="0.910000_0.910000_0.910000_0.000000_0.000000">
-                <texture />
-                <color rgba="0.91 0.91 0.91 1" />
-            </material>
-        </visual>
-        <visual>
-            <origin xyz="0.0345519 0.00182103 0.0272507" rpy="0 -0 0" />
-            <geometry>
-                <mesh filename="package://sentry_pkg/meshes/_1111_11.stl" scale="1 1 1" />
-            </geometry>
-            <material name="0.910000_0.910000_0.910000_0.000000_0.000000">
-                <texture />
-                <color rgba="0.91 0.91 0.91 1" />
-            </material>
-        </visual>
-        <visual>
-            <origin xyz="0.0345519 0.00182103 0.0272507" rpy="0 -0 0" />
-            <geometry>
-                <mesh filename="package://sentry_pkg/meshes/_1111_12.stl" scale="1 1 1" />
-            </geometry>
-            <material name="0.910000_0.910000_0.910000_0.000000_0.000000">
-                <texture />
-                <color rgba="0.91 0.91 0.91 1" />
-            </material>
-        </visual>
-        <visual>
-            <origin xyz="0.0345519 0.00182103 0.0272507" rpy="0 -0 0" />
-            <geometry>
-                <mesh filename="package://sentry_pkg/meshes/_1111_13.stl" scale="1 1 1" />
-            </geometry>
-            <material name="0.910000_0.910000_0.910000_0.000000_0.000000">
-                <texture />
-                <color rgba="0.91 0.91 0.91 1" />
-            </material>
-        </visual>
-        <visual>
-            <origin xyz="0.0345519 0.00182103 0.0272507" rpy="0 -0 0" />
-            <geometry>
-                <mesh filename="package://sentry_pkg/meshes/_1111_14.stl" scale="1 1 1" />
-            </geometry>
-            <material name="0.910000_0.910000_0.910000_0.000000_0.000000">
-                <texture />
-                <color rgba="0.91 0.91 0.91 1" />
-            </material>
-        </visual>
-        <visual>
-            <origin xyz="0.0345519 0.00182103 0.0272507" rpy="0 -0 0" />
-            <geometry>
-                <mesh filename="package://sentry_pkg/meshes/_1111_15.stl" scale="1 1 1" />
-            </geometry>
-            <material name="0.910000_0.910000_0.910000_0.000000_0.000000">
-                <texture />
-                <color rgba="0.91 0.91 0.91 1" />
-            </material>
-        </visual>
-        <visual>
-            <origin xyz="0.0345519 0.00182103 0.0272507" rpy="0 -0 0" />
-            <geometry>
-                <mesh filename="package://sentry_pkg/meshes/_1111_16.stl" scale="1 1 1" />
-            </geometry>
-            <material name="0.910000_0.910000_0.910000_0.000000_0.000000">
-                <texture />
-                <color rgba="0.91 0.91 0.91 1" />
-            </material>
-        </visual>
-        <visual>
-            <origin xyz="0.0345519 0.00182103 0.0272507" rpy="0 -0 0" />
-            <geometry>
-                <mesh filename="package://sentry_pkg/meshes/_1111_17.stl" scale="1 1 1" />
-            </geometry>
-            <material name="0.910000_0.910000_0.910000_0.000000_0.000000">
-                <texture />
-                <color rgba="0.91 0.91 0.91 1" />
-            </material>
-        </visual>
-        <visual>
-            <origin xyz="0.0345519 0.00182103 0.0272507" rpy="0 -0 0" />
-            <geometry>
-                <mesh filename="package://sentry_pkg/meshes/_1111_18.stl" scale="1 1 1" />
-            </geometry>
-            <material name="0.910000_0.910000_0.910000_0.000000_0.000000">
-                <texture />
-                <color rgba="0.91 0.91 0.91 1" />
-            </material>
-        </visual>
-        <visual>
-            <origin xyz="0.0345519 0.00182103 0.0272507" rpy="0 -0 0" />
-            <geometry>
-                <mesh filename="package://sentry_pkg/meshes/_1111_19.stl" scale="1 1 1" />
-            </geometry>
-            <material name="0.910000_0.910000_0.910000_0.000000_0.000000">
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