Commit message: pre ai

File: urdf/sentry.urdf.xacro (robot description, xacro)
@@ -1,70 +1,76 @@
+<?xml version="1.0"?>
 <!--URDF generated by ONSHAPE BY PTC INC, 1.217-->
-<robot name="assembly_3">
-    <link name="part_1">
-        <inertial>
-            <mass value="0.0701287" />
-            <origin xyz="1.20374e-17 2.46519e-32 0.126108" rpy="0 -0 0" />
-            <inertia ixx="0.00192346" ixy="0" ixz="0" iyy="0.00192346" iyz="0" izz="0.00310341" />
-        </inertial>
-        <visual>
-            <origin xyz="0 -1.82166e-17 0.0734155" rpy="0 -0 0" />
-            <geometry>
-                <mesh filename="package://assembly_3/meshes/Part_1.stl" scale="1 1 1" />
-            </geometry>
-            <material name="0.615686_0.811765_0.929412_0.000000_0.000000">
-                <color rgba="0.615686 0.811765 0.929412 1" />
-            </material>
-        </visual>
-    </link>
-    <link name="part_1_1">
-        <inertial>
-            <mass value="0.00421105" />
-            <origin xyz="0.00100261 -0.00244355 0.0730117" rpy="0 -0 2.48157" />
-            <inertia ixx="1.8557e-05" ixy="4.2327e-06" ixz="1.56708e-08" iyy="1.90292e-05" iyz="-3.81928e-08" izz="2.21682e-05" />
-        </inertial>
-        <visual>
-            <origin xyz="-1.68946e-18 -2.17675e-18 0" rpy="0 -0 2.48157" />
-            <geometry>
-                <mesh filename="package://assembly_3/meshes/Part_1_1.stl" scale="1 1 1" />
-            </geometry>
-            <material name="0.615686_0.811765_0.929412_0.000000_0.000000">
-                <color rgba="0.615686 0.811765 0.929412 1" />
-            </material>
-        </visual>
-    </link>
-    <link name="part_1_2">
-        <inertial>
-            <mass value="0.00018588" />
-            <origin xyz="-6.05411e-19 -4.2157e-19 0.02065" rpy="0 -0 0.608263" />
-            <inertia ixx="9.29949e-08" ixy="0" ixz="0" iyy="9.29949e-08" iyz="0" izz="1.33148e-07" />
-        </inertial>
-        <visual>
-            <origin xyz="1.3244e-18 -1.90196e-18 0" rpy="0 -0 0.608263" />
-            <geometry>
-                <mesh filename="package://assembly_3/meshes/Part_1_2.stl" scale="1 1 1" />
-            </geometry>
-            <material name="0.615686_0.811765_0.929412_0.000000_0.000000">
-                <color rgba="0.615686 0.811765 0.929412 1" />
-            </material>
-        </visual>
-    </link>
-    <link name="root" />
-    <joint name="fastened_1" type="fixed">
-        <origin xyz="0 1.38778e-17 -8.69386e-19" rpy="-1.5708 -0 3.14159" />
-        <axis xyz="0 0 -1" />
-        <parent link="root" />
-        <child link="part_1" />
-    </joint>
-    <joint name="headlink" type="continuous">
-        <origin xyz="3.00043e-17 -1.82344e-18 0.252215" rpy="0 -0 -3.14159" />
-        <axis xyz="0 0 -1" />
-        <parent link="part_1" />
-        <child link="part_1_1" />
-    </joint>
-    <joint name="lidar" type="continuous">
-        <origin xyz="0.0884778 -0.20163 0.0718" rpy="0 0 -0.660022" />
-        <axis xyz="0 0 -1" />
-        <parent link="part_1_1" />
-        <child link="part_1_2" />
-    </joint>
+<robot name="sentry">
+  <link name="part_1">
+    <inertial>
+      <mass value="0.0701287"/>
+      <origin xyz="1.20374e-17 2.46519e-32 0.126108" rpy="0 -0 0"/>
+      <inertia ixx="0.00192346" ixy="0" ixz="0" iyy="0.00192346" iyz="0" izz="0.00310341"/>
+    </inertial>
+    <visual>
+      <origin xyz="0 -1.82166e-17 0.0734155" rpy="0 -0 0"/>
+      <geometry>
+        <mesh filename="package://sentry_pkg/meshes/Part_1.stl" scale="1 1 1"/>
+      </geometry>
+      <material name="0.615686_0.811765_0.929412_0.000000_0.000000">
+        <color rgba="0.615686 0.811765 0.929412 1"/>
+      </material>
+    </visual>
+  </link>
+  <link name="part_1_1">
+    <inertial>
+      <mass value="0.00421105"/>
+      <origin xyz="0.00100261 -0.00244355 0.0730117" rpy="0 -0 2.48157"/>
+      <inertia ixx="1.8557e-05" ixy="4.2327e-06" ixz="1.56708e-08" iyy="1.90292e-05" iyz="-3.81928e-08" izz="2.21682e-05"/>
+    </inertial>
+    <visual>
+      <origin xyz="-1.68946e-18 -2.17675e-18 0" rpy="0 -0 2.48157"/>
+      <geometry>
+        <mesh filename="package://sentry_pkg/meshes/Part_1_1.stl" scale="1 1 1"/>
+      </geometry>
+      <material name="0.615686_0.811765_0.929412_0.000000_0.000000">
+        <color rgba="0.615686 0.811765 0.929412 1"/>
+      </material>
+    </visual>
+  </link>
+  <link name="part_1_2">
+    <inertial>
+      <mass value="0.00018588"/>
+      <origin xyz="-6.05411e-19 -4.2157e-19 0.02065" rpy="0 -0 0.608263"/>
+      <inertia ixx="9.29949e-08" ixy="0" ixz="0" iyy="9.29949e-08" iyz="0" izz="1.33148e-07"/>
+    </inertial>
+    <visual>
+      <origin xyz="1.3244e-18 -1.90196e-18 0" rpy="0 -0 0.608263"/>
+      <geometry>
+        <mesh filename="package://sentry_pkg/meshes/Part_1_2.stl" scale="1 1 1"/>
+      </geometry>
+      <material name="0.615686_0.811765_0.929412_0.000000_0.000000">
+        <color rgba="0.615686 0.811765 0.929412 1"/>
+      </material>
+    </visual>
+  </link>
+  <link name="root"/>
+  <joint name="fastened_1" type="fixed">
+    <origin xyz="0 1.38778e-17 -8.69386e-19" rpy="-1.5708 -0 3.14159"/>
+    <axis xyz="0 0 -1"/>
+    <parent link="root"/>
+    <child link="part_1"/>
+  </joint>
+  <joint name="headlink" type="continuous">
+    <origin xyz="3.00043e-17 -1.82344e-18 0.252215" rpy="0 -0 -3.14159"/>
+    <axis xyz="0 0 -1"/>
+    <parent link="part_1"/>
+    <child link="part_1_1"/>
+  </joint>
+  <joint name="lidar" type="continuous">
+    <origin xyz="0.0884778 -0.20163 0.0718" rpy="0 0 -0.660022"/>
+    <axis xyz="0 0 -1"/>
+    <parent link="part_1_1"/>
+    <child link="part_1_2"/>
+  </joint>
+  <gazebo>
+    <plugin name="gz::sim::systems::Physics" filename="gz-sim-physics-system"/>
+    <plugin name="gz::sim::systems::UserCommands" filename="gz-sim-user-commands-system"/>
+    <plugin name="gz::sim::systems::SceneBroadcaster" filename="gz-sim-scene-broadcaster-system"/>
+  </gazebo>
 </robot>

Commit message: updated model

File: urdf/sentry.urdf.xacro (robot description, xacro)
@@ -1,5 +1,5 @@
 <?xml version="1.0"?>
 <!--URDF generated by ONSHAPE BY PTC INC, 1.217-->
-<robot name="sentry">
+<robot name="sentry_pkg">
   <link name="part_1">
     <inertial>
@@ -20,10 +20,10 @@
   <link name="part_1_1">
     <inertial>
-      <mass value="0.00421105"/>
-      <origin xyz="0.00100261 -0.00244355 0.0730117" rpy="0 -0 2.48157"/>
-      <inertia ixx="1.8557e-05" ixy="4.2327e-06" ixz="1.56708e-08" iyy="1.90292e-05" iyz="-3.81928e-08" izz="2.21682e-05"/>
+      <mass value="0.00414744"/>
+      <origin xyz="-0.00211769 -0.00164536 0.0741316" rpy="0 -0 1.18195"/>
+      <inertia ixx="2.08028e-05" ixy="-3.50322e-06" ixz="-4.24357e-08" iyy="1.60288e-05" iyz="-3.29709e-08" izz="2.21034e-05"/>
     </inertial>
     <visual>
-      <origin xyz="-1.68946e-18 -2.17675e-18 0" rpy="0 -0 2.48157"/>
+      <origin xyz="-2.54975e-18 1.04465e-18 0" rpy="0 -0 1.18195"/>
       <geometry>
         <mesh filename="package://sentry_pkg/meshes/Part_1_1.stl" scale="1 1 1"/>
@@ -37,9 +37,9 @@
     <inertial>
       <mass value="0.00018588"/>
-      <origin xyz="-6.05411e-19 -4.2157e-19 0.02065" rpy="0 -0 0.608263"/>
+      <origin xyz="2.43997e-19 -6.96211e-19 0.02065" rpy="0 -0 1.90788"/>
       <inertia ixx="9.29949e-08" ixy="0" ixz="0" iyy="9.29949e-08" iyz="0" izz="1.33148e-07"/>
     </inertial>
     <visual>
-      <origin xyz="1.3244e-18 -1.90196e-18 0" rpy="0 -0 0.608263"/>
+      <origin xyz="2.18721e-18 7.6654e-19 0" rpy="0 -0 1.90788"/>
       <geometry>
         <mesh filename="package://sentry_pkg/meshes/Part_1_2.stl" scale="1 1 1"/>
@@ -58,5 +58,5 @@
   </joint>
   <joint name="headlink" type="continuous">
-    <origin xyz="3.00043e-17 -1.82344e-18 0.252215" rpy="0 -0 -3.14159"/>
+    <origin xyz="-2.83918e-18 3.04852e-18 0.252215" rpy="0 -0 3.14159"/>
     <axis xyz="0 0 -1"/>
     <parent link="part_1"/>
@@ -64,13 +64,8 @@
   </joint>
   <joint name="lidar" type="continuous">
-    <origin xyz="0.0884778 -0.20163 0.0718" rpy="0 0 -0.660022"/>
+    <origin xyz="-0.170562 -0.139254 0.0718" rpy="0 0 -1.95964"/>
     <axis xyz="0 0 -1"/>
     <parent link="part_1_1"/>
     <child link="part_1_2"/>
   </joint>
-  <gazebo>
-    <plugin name="gz::sim::systems::Physics" filename="gz-sim-physics-system"/>
-    <plugin name="gz::sim::systems::UserCommands" filename="gz-sim-user-commands-system"/>
-    <plugin name="gz::sim::systems::SceneBroadcaster" filename="gz-sim-scene-broadcaster-system"/>
-  </gazebo>
 </robot>

Commit message: good moodel

File: urdf/sentry.urdf.xacro (robot description, xacro)
@@ -2,5 +2,5 @@
 <!--URDF generated by ONSHAPE BY PTC INC, 1.217-->
 <robot name="sentry_pkg">
-  <link name="part_1">
+  <link name="body">
     <inertial>
       <mass value="0.0701287"/>
@@ -11,5 +11,5 @@
       <origin xyz="0 -1.82166e-17 0.0734155" rpy="0 -0 0"/>
       <geometry>
-        <mesh filename="package://sentry_pkg/meshes/Part_1.stl" scale="1 1 1"/>
+        <mesh filename="package://sentry_pkg/meshes/Body.stl" scale="1 1 1"/>
       </geometry>
       <material name="0.615686_0.811765_0.929412_0.000000_0.000000">
@@ -17,6 +17,12 @@
       </material>
     </visual>
+    <collision>
+      <origin xyz="0 0 0.01" rpy="0 0 0"/>
+      <geometry>
+        <box size="0.3 0.3 0.02"/>
+      </geometry>
+    </collision>
   </link>
-  <link name="part_1_1">
+  <link name="head">
     <inertial>
       <mass value="0.00414744"/>
@@ -27,5 +33,5 @@
       <origin xyz="-2.54975e-18 1.04465e-18 0" rpy="0 -0 1.18195"/>
       <geometry>
-        <mesh filename="package://sentry_pkg/meshes/Part_1_1.stl" scale="1 1 1"/>
+        <mesh filename="package://sentry_pkg/meshes/Head.stl" scale="1 1 1"/>
       </geometry>
       <material name="0.615686_0.811765_0.929412_0.000000_0.000000">
@@ -34,5 +40,5 @@
     </visual>
   </link>
-  <link name="part_1_2">
+  <link name="lidar">
     <inertial>
       <mass value="0.00018588"/>
@@ -43,5 +49,5 @@
       <origin xyz="2.18721e-18 7.6654e-19 0" rpy="0 -0 1.90788"/>
       <geometry>
-        <mesh filename="package://sentry_pkg/meshes/Part_1_2.stl" scale="1 1 1"/>
+        <mesh filename="package://sentry_pkg/meshes/Lidar.stl" scale="1 1 1"/>
       </geometry>
       <material name="0.615686_0.811765_0.929412_0.000000_0.000000">
@@ -51,21 +57,21 @@
   </link>
   <link name="root"/>
-  <joint name="fastened_1" type="fixed">
-    <origin xyz="0 1.38778e-17 -8.69386e-19" rpy="-1.5708 -0 3.14159"/>
+  <joint name="fastened_2" type="fixed">
+    <origin xyz="0 0 0" rpy="0 -0 3.14159"/>
     <axis xyz="0 0 -1"/>
     <parent link="root"/>
-    <child link="part_1"/>
+    <child link="body"/>
   </joint>
   <joint name="headlink" type="continuous">
-    <origin xyz="-2.83918e-18 3.04852e-18 0.252215" rpy="0 -0 3.14159"/>
+    <origin xyz="-2.54975e-18 5.65558e-17 0.252215" rpy="0 -0 3.14159"/>
     <axis xyz="0 0 -1"/>
-    <parent link="part_1"/>
-    <child link="part_1_1"/>
+    <parent link="body"/>
+    <child link="head"/>
   </joint>
-  <joint name="lidar" type="continuous">
+  <joint name="lidarlink" type="continuous">
     <origin xyz="-0.170562 -0.139254 0.0718" rpy="0 0 -1.95964"/>
     <axis xyz="0 0 -1"/>
-    <parent link="part_1_1"/>
-    <child link="part_1_2"/>
+    <parent link="head"/>
+    <child link="lidar"/>
   </joint>
 </robot>

Commit message: made base instaed of root

File: urdf/sentry.urdf.xacro (robot description, xacro)
@@ -2,4 +2,5 @@
 <!--URDF generated by ONSHAPE BY PTC INC, 1.217-->
 <robot name="sentry_pkg">
+  <link name="base_footprint"/>
   <link name="body">
     <inertial>
@@ -56,10 +57,8 @@
     </visual>
   </link>
-  <link name="root"/>
-  <joint name="fastened_2" type="fixed">
-    <origin xyz="0 0 0" rpy="0 -0 3.14159"/>
-    <axis xyz="0 0 -1"/>
-    <parent link="root"/>
+  <joint name="base_joint" type="fixed">
+    <parent link="base_footprint"/>
     <child link="body"/>
+    <origin xyz="0.0 0.0 0.0" rpy="0 0 0"/>
   </joint>
   <joint name="headlink" type="continuous">

Commit message: cleaned up some things to get slam to work

File: urdf/sentry.urdf.xacro (robot description, xacro)
@@ -68,7 +68,6 @@
     <child link="head"/>
   </joint>
-  <joint name="lidarlink" type="continuous">
+  <joint name="lidarlink" type="fixed">
     <origin xyz="-0.170562 -0.139254 0.0718" rpy="0 0 -1.95964"/>
-    <axis xyz="0 0 -1"/>
     <parent link="head"/>
     <child link="lidar"/>
@@ -78,5 +77,5 @@
       <always_on>true</always_on>
       <visualize>true</visualize>
-      <update_rate>5</update_rate>
+      <update_rate>10</update_rate>
       <topic>scan</topic>
       <gz_frame_id>lidar</gz_frame_id>

Commit message: added odo pods

File: urdf/sentry.urdf.xacro (robot description, xacro)
@@ -4,12 +4,12 @@
   <link name="body">
     <inertial>
-      <mass value="0.0701287"/>
-      <origin xyz="1.20374e-17 2.46519e-32 0.126108" rpy="0 -0 0"/>
-      <inertia ixx="0.00192346" ixy="0" ixz="0" iyy="0.00192346" iyz="0" izz="0.00310341"/>
+      <mass value="0.0507536"/>
+      <origin xyz="-2.33205e-05 -3.02404e-05 0.160359" rpy="0 -0 0"/>
+      <inertia ixx="0.00127958" ixy="3.57925e-11" ixz="-1.40827e-07" iyy="0.00127958" iyz="-1.82614e-07" izz="0.00226416"/>
     </inertial>
     <visual>
       <origin xyz="0 -1.82166e-17 0.0734155" rpy="0 -0 0"/>
       <geometry>
-        <mesh filename="package://sentry_pkg/meshes/Body.stl" scale="1 1 1"/>
+        <mesh filename="package://sentry_pkg/meshes/Body.gltf" scale="1 1 1"/>
       </geometry>
       <material name="0.615686_0.811765_0.929412_0.000000_0.000000">
@@ -17,10 +17,4 @@
       </material>
     </visual>
-    <collision>
-      <origin xyz="0 0 0.01" rpy="0 0 0"/>
-      <geometry>
-        <box size="0.3 0.3 0.02"/>
-      </geometry>
-    </collision>
   </link>
   <link name="head">
@@ -33,5 +27,5 @@
       <origin xyz="-2.54975e-18 1.04465e-18 0" rpy="0 -0 1.18195"/>
       <geometry>
-        <mesh filename="package://sentry_pkg/meshes/Head.stl" scale="1 1 1"/>
+        <mesh filename="package://sentry_pkg/meshes/Head.gltf" scale="1 1 1"/>
       </geometry>
       <material name="0.615686_0.811765_0.929412_0.000000_0.000000">
@@ -49,5 +43,37 @@
       <origin xyz="2.18721e-18 7.6654e-19 0" rpy="0 -0 1.90788"/>
       <geometry>
-        <mesh filename="package://sentry_pkg/meshes/Lidar.stl" scale="1 1 1"/>
+        <mesh filename="package://sentry_pkg/meshes/Lidar.gltf" scale="1 1 1"/>
+      </geometry>
+      <material name="0.615686_0.811765_0.929412_0.000000_0.000000">
+        <color rgba="0.615686 0.811765 0.929412 1"/>
+      </material>
+    </visual>
+  </link>
+  <link name="odowheel">
+    <inertial>
+      <mass value="3.2572e-05"/>
+      <origin xyz="0 0.009 4.67781e-19" rpy="0 -0 0"/>
+      <inertia ixx="5.56982e-09" ixy="0" ixz="0" iyy="9.38075e-09" iyz="0" izz="5.56982e-09"/>
+    </inertial>
+    <visual>
+      <origin xyz="0 0.009 -1.46958e-18" rpy="0 -0 0"/>
+      <geometry>
+        <mesh filename="package://sentry_pkg/meshes/OdoWheel.gltf" scale="1 1 1"/>
+      </geometry>
+      <material name="0.615686_0.811765_0.929412_0.000000_0.000000">
+        <color rgba="0.615686 0.811765 0.929412 1"/>
+      </material>
+    </visual>
+  </link>
+  <link name="odowheel_1">
+    <inertial>
+      <mass value="3.2572e-05"/>
+      <origin xyz="0 0.009 4.67781e-19" rpy="0 -0 0"/>
+      <inertia ixx="5.56982e-09" ixy="0" ixz="0" iyy="9.38075e-09" iyz="0" izz="5.56982e-09"/>
+    </inertial>
+    <visual>
+      <origin xyz="0 0.009 -1.46958e-18" rpy="0 -0 0"/>
+      <geometry>
+        <mesh filename="package://sentry_pkg/meshes/OdoWheel.gltf" scale="1 1 1"/>
       </geometry>
       <material name="0.615686_0.811765_0.929412_0.000000_0.000000">
@@ -57,7 +83,8 @@
   </link>
   <joint name="base_joint" type="fixed">
+    <origin xyz="0 0 0" rpy="0 -0 3.14159"/>
+    <axis xyz="-0 -0 -1"/>
     <parent link="base_footprint"/>
     <child link="body"/>
-    <origin xyz="0.0 0.0 0.0" rpy="0 0 0"/>
   </joint>
   <joint name="headlink" type="continuous">
@@ -67,8 +94,21 @@
     <child link="head"/>
   </joint>
-  <joint name="lidarlink" type="fixed">
+  <joint name="lidarlink" type="continuous">
     <origin xyz="-0.170562 -0.139254 0.0718" rpy="0 0 -1.95964"/>
+    <axis xyz="0 0 -1"/>
     <parent link="head"/>
     <child link="lidar"/>
+  </joint>
+  <joint name="odowheel_x" type="fixed">
+    <origin xyz="-0.089012 -0.009 0.0286405" rpy="3.14159 -0 3.14159"/>
+    <axis xyz="0 -1 0"/>
+    <parent link="body"/>
+    <child link="odowheel"/>
+  </joint>
+  <joint name="odowheel_y" type="fixed">
+    <origin xyz="0.014 -0.089012 0.0286405" rpy="0 0 -1.5708"/>
+    <axis xyz="0 -1 0"/>
+    <parent link="body"/>
+    <child link="odowheel_1"/>
   </joint>
   <gazebo reference="lidar">
@@ -101,11 +141,3 @@
     </sensor>
   </gazebo>
-  <gazebo>
-    <plugin filename="ignition-gazebo-odometry-publisher-system" name="ignition::gazebo::systems::OdometryPublisher">
-      <odom_frame>odom</odom_frame>
-      <robot_base_frame>base_footprint</robot_base_frame>
-      <odom_publish_frequency>50</odom_publish_frequency>
-      <dimensions>2</dimensions>
-    </plugin>
-  </gazebo>
 </robot>

Commit message: fixed wrong file format

File: urdf/sentry.urdf.xacro (robot description, xacro)
@@ -1,5 +1,5 @@
 <?xml version="1.0"?>
+<!--URDF generated by ONSHAPE BY PTC INC, 1.217-->
 <robot name="sentry_pkg">
-  <link name="base_footprint"/>
   <link name="body">
     <inertial>
@@ -11,5 +11,5 @@
       <origin xyz="0 -1.82166e-17 0.0734155" rpy="0 -0 0"/>
       <geometry>
-        <mesh filename="package://sentry_pkg/meshes/Body.gltf" scale="1 1 1"/>
+        <mesh filename="package://sentry_pkg/meshes/Body.stl" scale="1 1 1"/>
       </geometry>
       <material name="0.615686_0.811765_0.929412_0.000000_0.000000">
@@ -27,5 +27,5 @@
       <origin xyz="-2.54975e-18 1.04465e-18 0" rpy="0 -0 1.18195"/>
       <geometry>
-        <mesh filename="package://sentry_pkg/meshes/Head.gltf" scale="1 1 1"/>
+        <mesh filename="package://sentry_pkg/meshes/Head.stl" scale="1 1 1"/>
       </geometry>
       <material name="0.615686_0.811765_0.929412_0.000000_0.000000">
@@ -43,5 +43,5 @@
       <origin xyz="2.18721e-18 7.6654e-19 0" rpy="0 -0 1.90788"/>
       <geometry>
-        <mesh filename="package://sentry_pkg/meshes/Lidar.gltf" scale="1 1 1"/>
+        <mesh filename="package://sentry_pkg/meshes/Lidar.stl" scale="1 1 1"/>
       </geometry>
       <material name="0.615686_0.811765_0.929412_0.000000_0.000000">
@@ -59,5 +59,5 @@
       <origin xyz="0 0.009 -1.46958e-18" rpy="0 -0 0"/>
       <geometry>
-        <mesh filename="package://sentry_pkg/meshes/OdoWheel.gltf" scale="1 1 1"/>
+        <mesh filename="package://sentry_pkg/meshes/OdoWheel.stl" scale="1 1 1"/>
       </geometry>
       <material name="0.615686_0.811765_0.929412_0.000000_0.000000">
@@ -65,4 +65,10 @@
       </material>
     </visual>
+    <collision>
+      <origin xyz="0 0 0" rpy="1.5707 0 0"/>
+      <geometry>
+        <cylinder radius="0.024" length="0.018"/>
+      </geometry>
+    </collision>
   </link>
   <link name="odowheel_1">
@@ -75,5 +81,5 @@
       <origin xyz="0 0.009 -1.46958e-18" rpy="0 -0 0"/>
       <geometry>
-        <mesh filename="package://sentry_pkg/meshes/OdoWheel.gltf" scale="1 1 1"/>
+        <mesh filename="package://sentry_pkg/meshes/OdoWheel.stl" scale="1 1 1"/>
       </geometry>
       <material name="0.615686_0.811765_0.929412_0.000000_0.000000">
@@ -81,9 +87,16 @@
       </material>
     </visual>
+    <collision>
+      <origin xyz="0 0 0" rpy="1.5707 0 0"/>
+      <geometry>
+        <cylinder radius="0.024" length="0.018"/>
+      </geometry>
+    </collision>
   </link>
-  <joint name="base_joint" type="fixed">
+  <link name="root"/>
+  <joint name="fastened_2" type="fixed">
     <origin xyz="0 0 0" rpy="0 -0 3.14159"/>
     <axis xyz="-0 -0 -1"/>
-    <parent link="base_footprint"/>
+    <parent link="root"/>
     <child link="body"/>
   </joint>

Commit message: added body collsion

File: urdf/sentry.urdf.xacro (robot description, xacro)
@@ -17,4 +17,10 @@
       </material>
     </visual>
+    <collision>
+      <origin xyz="0 0 0" rpy="0 0 0"/>
+      <geometry>
+        <cylinder radius="0.03" length="0.01"/>
+      </geometry>
+    </collision>
   </link>
   <link name="head">

Commit message: working odom no lidar

File: urdf/sentry.urdf.xacro (robot description, xacro)
@@ -113,11 +113,10 @@
     <child link="head"/>
   </joint>
-  <joint name="lidarlink" type="continuous">
+  <joint name="lidarlink" type="fixed">
     <origin xyz="-0.170562 -0.139254 0.0718" rpy="0 0 -1.95964"/>
-    <axis xyz="0 0 -1"/>
     <parent link="head"/>
     <child link="lidar"/>
   </joint>
-  <joint name="odowheel_x" type="fixed">
+  <joint name="odowheel_x" type="continuous">
     <origin xyz="-0.089012 -0.009 0.0286405" rpy="3.14159 -0 3.14159"/>
     <axis xyz="0 -1 0"/>
@@ -125,5 +124,5 @@
     <child link="odowheel"/>
   </joint>
-  <joint name="odowheel_y" type="fixed">
+  <joint name="odowheel_y" type="continuous">
     <origin xyz="0.014 -0.089012 0.0286405" rpy="0 0 -1.5708"/>
     <axis xyz="0 -1 0"/>
@@ -160,3 +159,18 @@
     </sensor>
   </gazebo>
+  <gazebo>
+    <plugin filename="ignition-gazebo-odometry-publisher-system" name="ignition::gazebo::systems::OdometryPublisher">
+      <odom_frame>odom</odom_frame>
+      <robot_base_frame>root</robot_base_frame>
+      <publish_odom_tf>true</publish_odom_tf>
+      <dimensions>3</dimensions>
+    </plugin>
+    <plugin filename="ignition-gazebo-joint-state-publisher-system" name="ignition::gazebo::systems::JointStatePublisher">
+    </plugin>
+  </gazebo>
+  <gazebo>
+    <plugin filename="ignition-gazebo-joint-state-publisher-system" name="ignition::gazebo::systems::JointStatePublisher">
+      <joint_name>headlink</joint_name>
+    </plugin>
+  </gazebo>
 </robot>

Commit message: fixed sim

File: urdf/sentry.urdf.xacro (robot description, xacro)
@@ -39,4 +39,9 @@
       </material>
     </visual>
+    <collision>
+      <geometry>
+        <mesh filename="package://sentry_pkg/meshes/Head.stl" scale="1 1 1"/>
+      </geometry>
+    </collision>
   </link>
   <link name="lidar">
@@ -165,4 +170,7 @@
       <publish_odom_tf>true</publish_odom_tf>
       <dimensions>3</dimensions>
+      <ros>
+        <argument>-p use_sim_time:=true</argument>
+      </ros>
     </plugin>
     <plugin filename="ignition-gazebo-joint-state-publisher-system" name="ignition::gazebo::systems::JointStatePublisher">
@@ -170,4 +178,7 @@
       <joint_name>odowheel_x</joint_name>
       <joint_name>odowheel_y</joint_name>
+      <ros>
+        <argument>-p use_sim_time:=true</argument>
+      </ros>
     </plugin>
   </gazebo>
