Commit message: Rename sentry_pkg to thornbots_pkg, plus pending local work
Follows the GitHub repo rename Thornbots/sentry_pkg -> Thornbots/thornbots_pkg:
package name, module path and share directory all move.

This repo also had uncommitted work sitting in the tree, so it goes in with the
rename rather than being split out.

UNTESTED: the rename itself builds, the rest of this commit was never run.

Co-Authored-By: Claude Opus 5 (1M context) <noreply@anthropic.com>

File: urdf/sentry.urdf.xacro (robot description, xacro)
@@ -1,5 +1,5 @@
 <?xml version="1.0"?>
 <!--URDF generated by ONSHAPE BY PTC INC, 1.217-->
-<robot name="sentry_pkg">
+<robot name="thornbots_pkg">
   <link name="body">
     <inertial>
@@ -11,5 +11,5 @@
       <origin xyz="0 -1.82166e-17 0.0734155" rpy="0 -0 0"/>
       <geometry>
-        <mesh filename="package://sentry_pkg/meshes/Body.stl" scale="1 1 1"/>
+        <mesh filename="package://thornbots_pkg/meshes/Body.stl" scale="1 1 1"/>
       </geometry>
       <material name="0.615686_0.811765_0.929412_0.000000_0.000000">
@@ -27,5 +27,5 @@
       <origin xyz="-2.54975e-18 1.04465e-18 0" rpy="0 -0 1.18195"/>
       <geometry>
-        <mesh filename="package://sentry_pkg/meshes/Head.stl" scale="1 1 1"/>
+        <mesh filename="package://thornbots_pkg/meshes/Head.stl" scale="1 1 1"/>
       </geometry>
       <material name="0.615686_0.811765_0.929412_0.000000_0.000000">
@@ -43,5 +43,5 @@
       <origin xyz="2.18721e-18 7.6654e-19 0" rpy="0 -0 1.90788"/>
       <geometry>
-        <mesh filename="package://sentry_pkg/meshes/Lidar.stl" scale="1 1 1"/>
+        <mesh filename="package://thornbots_pkg/meshes/Lidar.stl" scale="1 1 1"/>
       </geometry>
       <material name="0.615686_0.811765_0.929412_0.000000_0.000000">
@@ -87,5 +87,5 @@
       <origin xyz="0 0.009 -1.46958e-18" rpy="0 -0 0"/>
       <geometry>
-        <mesh filename="package://sentry_pkg/meshes/OdoWheel.stl" scale="1 1 1"/>
+        <mesh filename="package://thornbots_pkg/meshes/OdoWheel.stl" scale="1 1 1"/>
       </geometry>
       <material name="0.615686_0.811765_0.929412_0.000000_0.000000">
@@ -103,5 +103,5 @@
       <origin xyz="0 0.009 -1.46958e-18" rpy="0 -0 0"/>
       <geometry>
-        <mesh filename="package://sentry_pkg/meshes/OdoWheel.stl" scale="1 1 1"/>
+        <mesh filename="package://thornbots_pkg/meshes/OdoWheel.stl" scale="1 1 1"/>
       </geometry>
       <material name="0.615686_0.811765_0.929412_0.000000_0.000000">

Commit message: URDF moves to sentry_v2; lidar_self_filter's sector from its CAD
urdf/sentry.urdf.xacro now describes the new sentry: sim's generated
sentry_v2 frames and meshes (meshes/sentry_v2/, coloured), with the wheel
and suspension joints fixed because /joint_states only carries headlink
and headpitch. Before, rviz showed the carriers and wheels with no
transform. It adds a muzzle frame on head_pitch at (0, 0.1128, 0): on the
pitch axis between the two stacked flywheels, from the CAD. The old
meshes go. The CV stack gets the camera from TF, so it follows this
file with no code change.

lidar_self_filter defaults to 0.09-1.41 rad (5-81 deg CCW from the gun).
Slicing the CAD at the RPLIDAR's scan plane (z 0.355 m, +-6 mm), the
gimbal, shooter and the lidar's own cover block 6-80 deg over the full
pitch range, and nothing on the chassis reaches the plane. Unverified on
hardware: the real lidar's 0 deg direction relative to the gun has not
been measured.

Co-Authored-By: Claude Opus 5.5 (1M context) <noreply@anthropic.com>

File: urdf/sentry.urdf.xacro (robot description, xacro)
@@ -1,159 +1,175 @@
 <?xml version="1.0"?>
-<!--URDF generated by ONSHAPE BY PTC INC, 1.217-->
-<robot name="thornbots_pkg">
-  <link name="body">
-    <inertial>
-      <mass value="0.0507536"/>
-      <origin xyz="-2.33205e-05 -3.02404e-05 0.160359" rpy="0 -0 0"/>
-      <inertia ixx="0.00127958" ixy="3.57925e-11" ixz="-1.40827e-07" iyy="0.00127958" iyz="-1.82614e-07" izz="0.00226416"/>
-    </inertial>
+<!-- The sentry as robot_state_publisher publishes it: sim/urdf/sentry_v2/sentry_v2.urdf's
+     frames and meshes, with the wheel and suspension joints fixed because
+     /joint_states only carries headlink and headpitch. sim's
+     test_urdf_constants.py pins the chain to the sim model. -->
+<robot name="sentry">
+  <link name="root">
     <visual>
-      <origin xyz="0 -1.82166e-17 0.0734155" rpy="0 -0 0"/>
       <geometry>
-        <mesh filename="package://thornbots_pkg/meshes/Body.stl" scale="1 1 1"/>
+        <mesh filename="package://thornbots_pkg/meshes/sentry_v2/root.stl"/>
       </geometry>
-      <material name="0.615686_0.811765_0.929412_0.000000_0.000000">
-        <color rgba="1 0 0 1"/>
-      </material>
+      <material name="root"><color rgba="0.18 0.18 0.2 1"/></material>
     </visual>
   </link>
+  <link name="body"/>
+  <joint name="fastened_2" type="fixed">
+    <parent link="root"/>
+    <child link="body"/>
+    <origin xyz="0 0 0" rpy="0 0 0"/>
+  </joint>
   <link name="head">
-    <inertial>
-      <mass value="0.00414744"/>
-      <origin xyz="-0.00211769 -0.00164536 0.0741316" rpy="0 -0 1.18195"/>
-      <inertia ixx="2.08028e-05" ixy="-3.50322e-06" ixz="-4.24357e-08" iyy="1.60288e-05" iyz="-3.29709e-08" izz="2.21034e-05"/>
-    </inertial>
     <visual>
-      <origin xyz="-2.54975e-18 1.04465e-18 0" rpy="0 -0 1.18195"/>
       <geometry>
-        <mesh filename="package://thornbots_pkg/meshes/Head.stl" scale="1 1 1"/>
+        <mesh filename="package://thornbots_pkg/meshes/sentry_v2/head.stl"/>
       </geometry>
-      <material name="0.615686_0.811765_0.929412_0.000000_0.000000">
-        <color rgba="1 0 0 1"/>
-      </material>
+      <material name="head"><color rgba="0.75 0.08 0.08 1"/></material>
     </visual>
   </link>
-  <link name="lidar">
-    <inertial>
-      <mass value="0.00018588"/>
-      <origin xyz="2.43997e-19 -6.96211e-19 0.02065" rpy="0 -0 1.90788"/>
-      <inertia ixx="9.29949e-08" ixy="0" ixz="0" iyy="9.29949e-08" iyz="0" izz="1.33148e-07"/>
-    </inertial>
+  <joint name="headlink" type="continuous">
+    <parent link="body"/>
+    <child link="head"/>
+    <origin xyz="-0.000171242 9.52126e-05 0.248293" rpy="0 0 0"/>
+    <axis xyz="-0 -0 -1"/>
+  </joint>
+  <link name="head_pitch">
     <visual>
-      <origin xyz="2.18721e-18 7.6654e-19 0" rpy="0 -0 1.90788"/>
       <geometry>
-        <mesh filename="package://thornbots_pkg/meshes/Lidar.stl" scale="1 1 1"/>
+        <mesh filename="package://thornbots_pkg/meshes/sentry_v2/head_pitch.stl"/>
       </geometry>
-      <material name="0.615686_0.811765_0.929412_0.000000_0.000000">
-        <color rgba="1 0 0 1"/>
-      </material>
+      <material name="head_pitch"><color rgba="0.9 0.35 0.1 1"/></material>
     </visual>
   </link>
-  <!-- Pitch stage for the head, so a camera mounted on it can tilt
-       independently of the yaw-only headlink joint below. No mesh of its
-       own, just a bare kinematic link the camera is fastened to. -->
-  <link name="head_pitch">
-    <inertial>
-      <mass value="0.005"/>
-      <origin xyz="0 0 0" rpy="0 0 0"/>
-      <inertia ixx="1e-06" ixy="0" ixz="0" iyy="1e-06" iyz="0" izz="1e-06"/>
-    </inertial>
-  </link>
-  <!-- Approximates a RealSense D435 (90x25x25mm, 72g); no mesh exists for
-       it yet so a plain box visual stands in until one is added. -->
-  <link name="camera">
-    <inertial>
-      <mass value="0.072"/>
-      <origin xyz="0 0 0" rpy="0 0 0"/>
-      <inertia ixx="1.05e-05" ixy="0" ixz="0" iyy="5.4e-05" iyz="0" izz="5.4e-05"/>
-    </inertial>
+  <joint name="headpitch" type="revolute">
+    <parent link="head"/>
+    <child link="head_pitch"/>
+    <origin xyz="-0.00760542 -0.100122 0.14235" rpy="0 0 0"/>
+    <axis xyz="0 1 0"/>
+    <limit lower="-0.6" upper="0.6" effort="200" velocity="10"/>
+  </joint>
+  <link name="carrier_0">
     <visual>
-      <origin xyz="0 0 0" rpy="0 0 0"/>
       <geometry>
-        <box size="0.025 0.09 0.025"/>
+        <mesh filename="package://thornbots_pkg/meshes/sentry_v2/carrier_0.stl"/>
       </geometry>
-      <material name="0.1_0.1_0.1_0.000000_0.000000">
-        <color rgba="0.1 0.1 0.1 1"/>
-      </material>
+      <material name="carrier_0"><color rgba="0.6 0.62 0.65 1"/></material>
     </visual>
   </link>
-  <link name="odowheel">
-    <inertial>
-      <mass value="3.2572e-05"/>
-      <origin xyz="0 0.009 4.67781e-19" rpy="0 -0 0"/>
-      <inertia ixx="5.56982e-09" ixy="0" ixz="0" iyy="9.38075e-09" iyz="0" izz="5.56982e-09"/>
-    </inertial>
+  <joint name="suspension_0" type="fixed">
+    <parent link="body"/>
+    <child link="carrier_0"/>
+    <origin xyz="6.61834e-09 -0.247 0.0954" rpy="0 0 0"/>
+  </joint>
+  <link name="wheel_0">
     <visual>
-      <origin xyz="0 0.009 -1.46958e-18" rpy="0 -0 0"/>
       <geometry>
-        <mesh filename="package://thornbots_pkg/meshes/OdoWheel.stl" scale="1 1 1"/>
+        <mesh filename="package://thornbots_pkg/meshes/sentry_v2/wheel_0.stl"/>
       </geometry>
-      <material name="0.615686_0.811765_0.929412_0.000000_0.000000">
-        <color rgba="1 0 0 1"/>
-      </material>
+      <material name="wheel_0"><color rgba="0.08 0.08 0.08 1"/></material>
     </visual>
   </link>
-  <link name="odowheel_1">
-    <inertial>
-      <mass value="3.2572e-05"/>
-      <origin xyz="0 0.009 4.67781e-19" rpy="0 -0 0"/>
-      <inertia ixx="5.56982e-09" ixy="0" ixz="0" iyy="9.38075e-09" iyz="0" izz="5.56982e-09"/>
-    </inertial>
+  <joint name="wheel_0_spin" type="fixed">
+    <parent link="carrier_0"/>
+    <child link="wheel_0"/>
+    <origin xyz="0 0 0" rpy="0 0 0"/>
+  </joint>
+  <link name="carrier_1">
     <visual>
-      <origin xyz="0 0.009 -1.46958e-18" rpy="0 -0 0"/>
       <geometry>
-        <mesh filename="package://thornbots_pkg/meshes/OdoWheel.stl" scale="1 1 1"/>
+        <mesh filename="package://thornbots_pkg/meshes/sentry_v2/carrier_1.stl"/>
       </geometry>
-      <material name="0.615686_0.811765_0.929412_0.000000_0.000000">
-        <color rgba="1 0 0 1"/>
-      </material>
+      <material name="carrier_1"><color rgba="0.6 0.62 0.65 1"/></material>
     </visual>
   </link>
-  <link name="root"/>
-  <joint name="fastened_2" type="fixed">
-    <origin xyz="0 0 0" rpy="0 -0 3.14159"/>
-    <parent link="root"/>
-    <child link="body"/>
+  <joint name="suspension_1" type="fixed">
+    <parent link="body"/>
+    <child link="carrier_1"/>
+    <origin xyz="0.247 6.61834e-09 0.0954" rpy="0 0 0"/>
   </joint>
-  <joint name="headlink" type="continuous">
-    <origin xyz="-2.54975e-18 5.65558e-17 0.252215" rpy="0 -0 3.14159"/>
-    <axis xyz="0 0 -1"/>
+  <link name="wheel_1">
+    <visual>
+      <geometry>
+        <mesh filename="package://thornbots_pkg/meshes/sentry_v2/wheel_1.stl"/>
+      </geometry>
+      <material name="wheel_1"><color rgba="0.08 0.08 0.08 1"/></material>
+    </visual>
+  </link>
+  <joint name="wheel_1_spin" type="fixed">
+    <parent link="carrier_1"/>
+    <child link="wheel_1"/>
+    <origin xyz="0 0 0" rpy="0 0 0"/>
+  </joint>
+  <link name="carrier_2">
+    <visual>
+      <geometry>
+        <mesh filename="package://thornbots_pkg/meshes/sentry_v2/carrier_2.stl"/>
+      </geometry>
+      <material name="carrier_2"><color rgba="0.6 0.62 0.65 1"/></material>
+    </visual>
+  </link>
+  <joint name="suspension_2" type="fixed">
     <parent link="body"/>
-    <child link="head"/>
+    <child link="carrier_2"/>
+    <origin xyz="-6.61834e-09 0.247 0.0954" rpy="0 0 0"/>
   </joint>
+  <link name="wheel_2">
+    <visual>
+      <geometry>
+        <mesh filename="package://thornbots_pkg/meshes/sentry_v2/wheel_2.stl"/>
+      </geometry>
+      <material name="wheel_2"><color rgba="0.08 0.08 0.08 1"/></material>
+    </visual>
+  </link>
+  <joint name="wheel_2_spin" type="fixed">
+    <parent link="carrier_2"/>
+    <child link="wheel_2"/>
+    <origin xyz="0 0 0" rpy="0 0 0"/>
+  </joint>
+  <link name="carrier_3">
+    <visual>
+      <geometry>
+        <mesh filename="package://thornbots_pkg/meshes/sentry_v2/carrier_3.stl"/>
+      </geometry>
+      <material name="carrier_3"><color rgba="0.6 0.62 0.65 1"/></material>
+    </visual>
+  </link>
+  <joint name="suspension_3" type="fixed">
+    <parent link="body"/>
+    <child link="carrier_3"/>
+    <origin xyz="-0.247 -6.61834e-09 0.0954" rpy="0 0 0"/>
+  </joint>
+  <link name="wheel_3">
+    <visual>
+      <geometry>
+        <mesh filename="package://thornbots_pkg/meshes/sentry_v2/wheel_3.stl"/>
+      </geometry>
+      <material name="wheel_3"><color rgba="0.08 0.08 0.08 1"/></material>
+    </visual>
+  </link>
+  <joint name="wheel_3_spin" type="fixed">
+    <parent link="carrier_3"/>
+    <child link="wheel_3"/>
+    <origin xyz="0 0 0" rpy="0 0 0"/>
+  </joint>
+  <link name="lidar"/>
   <joint name="lidarlink" type="fixed">
-    <origin xyz="-0.170562 -0.139254 0.0718" rpy="0 0 -1.95964"/>
     <parent link="head"/>
     <child link="lidar"/>
+    <origin xyz="-0.119391 -0.18501 0.0968001" rpy="0 0 0"/>
   </joint>
-  <!-- Pitch axis for the head-mounted camera. Centered laterally (y=0) at
-       the same height as the lidar's mount z (raised ~5cm to clear it),
-       moved forward (+x) from head center so it sits out past the head's
-       front face rather than buried inside it. rpy z tuned empirically
-       against the rendered scene/camera feed (head's own <visual> mesh
-       rotation is rpy="0 0 1.18195"; this is that value minus pi/2. A
-       subsequent 180deg flip turned out to be wrong too, so this is
-       back to that original value). -->
-  <joint name="headpitch" type="revolute">
-    <origin xyz="0.1 0 0.1218" rpy="0 0 -0.38885"/>
-    <axis xyz="0 1 0"/>
-    <parent link="head"/>
-    <child link="head_pitch"/>
-    <limit lower="-0.6" upper="0.6" effort="5" velocity="3"/>
-  </joint>
+  <link name="camera"/>
   <joint name="cameralink" type="fixed">
-    <origin xyz="0 0 0" rpy="0 0 0"/>
     <parent link="head_pitch"/>
     <child link="camera"/>
+    <origin xyz="0.0920381 0.0948673 0.0566588" rpy="0 0 0"/>
   </joint>
-  <joint name="odowheel_x" type="fixed">
-    <origin xyz="-0.089012 -0.009 0.0286405" rpy="3.14159 -0 3.14159"/>
-    <parent link="body"/>
-    <child link="odowheel"/>
-  </joint>
-  <joint name="odowheel_y" type="fixed">
-    <origin xyz="0.014 -0.089012 0.0286405" rpy="0 0 -1.5708"/>
-    <parent link="body"/>
-    <child link="odowheel_1"/>
+  <!-- Where the shot leaves: on the pitch axis, between the flywheels
+       (sentry_v2 CAD), pointing along head_pitch +x. Not in the generated
+       model; sim/urdf/sentry_v2.urdf.xacro adds the same frame. -->
+  <link name="muzzle"/>
+  <joint name="muzzlelink" type="fixed">
+    <parent link="head_pitch"/>
+    <child link="muzzle"/>
+    <origin xyz="0 0.1128 0" rpy="0 0 0"/>
   </joint>
 </robot>

Commit message: URDF: armor_0..3 frames, as sim's sentry_v2 has them
Four fixed frames on root at the armor faces from the CAD: origin at the
face centre, +x the outward normal (canted 15 deg up), +y horizontal,
drawn as a 135 x 125 mm box (the Small Armor Module, the only size in
ARCC 2026). sim's test_urdf_constants.py pins them to sim's model.

Co-Authored-By: Claude Opus 5.5 (1M context) <noreply@anthropic.com>

File: urdf/sentry.urdf.xacro (robot description, xacro)
@@ -151,4 +151,52 @@
     <child link="wheel_3"/>
     <origin xyz="0 0 0" rpy="0 0 0"/>
+  </joint>
+  <!-- Armor faces from the CAD, as sim/urdf/sentry_v2/sentry_v2.urdf generates them:
+       origin at the face centre, +x the outward normal (canted 15 deg up), +y
+       horizontal. The face is 0.135 (y) by 0.125 (z) m: the Small Armor
+       Module, the only size in ARCC 2026. -->
+  <link name="armor_0">
+    <visual>
+      <geometry><box size="0.003 0.135 0.125"/></geometry>
+      <material name="armor"><color rgba="0.85 0.85 0.85 1"/></material>
+    </visual>
+  </link>
+  <joint name="armor_0link" type="fixed">
+    <parent link="root"/>
+    <child link="armor_0"/>
+    <origin xyz="0.178162 0.178426 0.230361" rpy="0 -0.261856 0.785329"/>
+  </joint>
+  <link name="armor_1">
+    <visual>
+      <geometry><box size="0.003 0.135 0.125"/></geometry>
+      <material name="armor"><color rgba="0.85 0.85 0.85 1"/></material>
+    </visual>
+  </link>
+  <joint name="armor_1link" type="fixed">
+    <parent link="root"/>
+    <child link="armor_1"/>
+    <origin xyz="-0.177935 0.177863 0.135661" rpy="0 -0.261856 2.35613"/>
+  </joint>
+  <link name="armor_2">
+    <visual>
+      <geometry><box size="0.003 0.135 0.125"/></geometry>
+      <material name="armor"><color rgba="0.85 0.85 0.85 1"/></material>
+    </visual>
+  </link>
+  <joint name="armor_2link" type="fixed">
+    <parent link="root"/>
+    <child link="armor_2"/>
+    <origin xyz="-0.178505 -0.178235 0.230361" rpy="0 -0.261856 -2.35627"/>
+  </joint>
+  <link name="armor_3">
+    <visual>
+      <geometry><box size="0.003 0.135 0.125"/></geometry>
+      <material name="armor"><color rgba="0.85 0.85 0.85 1"/></material>
+    </visual>
+  </link>
+  <joint name="armor_3link" type="fixed">
+    <parent link="root"/>
+    <child link="armor_3"/>
+    <origin xyz="0.177593 -0.177673 0.135661" rpy="0 -0.261856 -0.785464"/>
   </joint>
   <link name="lidar"/>

Commit message: Chassis yaw as a joint under a heading-fixed root
RobotPose.chassis_yaw goes out as the URDF's new chassis_yaw joint
(root -> body, about -z like headlink). The head and the armor frames
re-parent: headlink hangs off root at the MCB's world head yaw, so
root->lidar and root->camera don't depend on chassis yaw, and armor_k
turns with body. odom->root carries no yaw, as rf2o's fixed_heading and
the EKF assume. README.md has why this isn't a body-fixed base_link.

Co-Authored-By: Claude Opus 5.5 (1M context) <noreply@anthropic.com>

File: urdf/sentry.urdf.xacro (robot description, xacro)
@@ -2,6 +2,10 @@
 <!-- The sentry as robot_state_publisher publishes it: sim/urdf/sentry_v2/sentry_v2.urdf's
      frames and meshes, with the wheel and suspension joints fixed because
-     /joint_states only carries headlink and headpitch. sim's
-     test_urdf_constants.py pins the chain to the sim model. -->
+     /joint_states only carries chassis_yaw, headlink and headpitch. sim's
+     test_urdf_constants.py pins the chain to the sim model.
+     root is heading-fixed (odom->root carries no yaw): the chassis turns
+     under it on chassis_yaw, and the head hangs off root with headlink at
+     the MCB's world head yaw, so lidar and camera never see chassis yaw.
+     The yaw bearing sits 0.2 mm off root's z axis; that offset is ignored. -->
 <robot name="sentry">
   <link name="root">
@@ -14,8 +18,9 @@
   </link>
   <link name="body"/>
-  <joint name="fastened_2" type="fixed">
+  <joint name="chassis_yaw" type="continuous">
     <parent link="root"/>
     <child link="body"/>
     <origin xyz="0 0 0" rpy="0 0 0"/>
+    <axis xyz="-0 -0 -1"/>
   </joint>
   <link name="head">
@@ -28,5 +33,5 @@
   </link>
   <joint name="headlink" type="continuous">
-    <parent link="body"/>
+    <parent link="root"/>
     <child link="head"/>
     <origin xyz="-0.000171242 9.52126e-05 0.248293" rpy="0 0 0"/>
@@ -163,5 +168,5 @@
   </link>
   <joint name="armor_0link" type="fixed">
-    <parent link="root"/>
+    <parent link="body"/>
     <child link="armor_0"/>
     <origin xyz="0.178162 0.178426 0.230361" rpy="0 -0.261856 0.785329"/>
@@ -174,5 +179,5 @@
   </link>
   <joint name="armor_1link" type="fixed">
-    <parent link="root"/>
+    <parent link="body"/>
     <child link="armor_1"/>
     <origin xyz="-0.177935 0.177863 0.135661" rpy="0 -0.261856 2.35613"/>
@@ -185,5 +190,5 @@
   </link>
   <joint name="armor_2link" type="fixed">
-    <parent link="root"/>
+    <parent link="body"/>
     <child link="armor_2"/>
     <origin xyz="-0.178505 -0.178235 0.230361" rpy="0 -0.261856 -2.35627"/>
@@ -196,5 +201,5 @@
   </link>
   <joint name="armor_3link" type="fixed">
-    <parent link="root"/>
+    <parent link="body"/>
     <child link="armor_3"/>
     <origin xyz="0.177593 -0.177673 0.135661" rpy="0 -0.261856 -0.785464"/>

Commit message: URDF: headlink and chassis_yaw turn about +z, so TF yaw == RobotPose.head_yaw
The MCB reports head_yaw CCW-positive (bag run00029, 2026-10-03: hand turns CCW
raised it). pose_translator publishes it unchanged as the joint position, and
the -z axis made root->head yaw = -head_yaw: camera and targets at the mirrored
bearing, aim point ~2x the gimbal angle off. No CV node negated head_yaw, so
nothing else compensated.

Tests (isaac_ros_jazzy_container, pytest test/): 72 passed. colcon build
thornbots_pkg ok; xacro shows axis 0 0 1.

Co-Authored-By: Claude Sonnet 5.5 <noreply@anthropic.com>

File: urdf/sentry.urdf.xacro (robot description, xacro)
@@ -22,5 +22,5 @@
     <child link="body"/>
     <origin xyz="0 0 0" rpy="0 0 0"/>
-    <axis xyz="-0 -0 -1"/>
+    <axis xyz="0 0 1"/>
   </joint>
   <link name="head">
@@ -36,5 +36,5 @@
     <child link="head"/>
     <origin xyz="-0.000171242 9.52126e-05 0.248293" rpy="0 0 0"/>
-    <axis xyz="-0 -0 -1"/>
+    <axis xyz="0 0 1"/>
   </joint>
   <link name="head_pitch">
