Commit message: added lidar back spinning

File: urdf/sentry.urdf.xacro (robot description, xacro)
@@ -119,6 +119,7 @@
     <child link="head"/>
   </joint>
-  <joint name="lidarlink" type="fixed">
+  <joint name="lidarlink" type="continuous">
     <origin xyz="-0.170562 -0.139254 0.0718" rpy="0 0 -1.95964"/>
+    <axis xyz="0 0 1"/>
     <parent link="head"/>
     <child link="lidar"/>

Commit message: removed last commit i tinhk roguhtly

File: urdf/sentry.urdf.xacro (robot description, xacro)
@@ -119,7 +119,6 @@
     <child link="head"/>
   </joint>
-  <joint name="lidarlink" type="continuous">
+  <joint name="lidarlink" type="fixed">
     <origin xyz="-0.170562 -0.139254 0.0718" rpy="0 0 -1.95964"/>
-    <axis xyz="0 0 1"/>
     <parent link="head"/>
     <child link="lidar"/>

Commit message: reads pose_data now
doesnt get exact ros formatted odom data from sim now it gets the same pose data as it would with real sensors

File: urdf/sentry.urdf.xacro (robot description, xacro)
@@ -17,10 +17,4 @@
       </material>
     </visual>
-    <collision>
-      <origin xyz="0 0 0" rpy="0 0 0"/>
-      <geometry>
-        <cylinder radius="0.03" length="0.01"/>
-      </geometry>
-    </collision>
   </link>
   <link name="head">
@@ -39,10 +33,4 @@
       </material>
     </visual>
-    <collision>
-      <origin xyz="-0.00211769 -0.00164536 0.0741316" rpy="0 -0 1.18195"/>
-      <geometry>
-        <box size="0.2 0.14 0.16075"/>
-      </geometry>
-    </collision>
   </link>
   <link name="lidar">
@@ -77,10 +65,4 @@
       </material>
     </visual>
-    <collision>
-      <origin xyz="0 0 0" rpy="1.5707 0 0"/>
-      <geometry>
-        <cylinder radius="0.024" length="0.018"/>
-      </geometry>
-    </collision>
   </link>
   <link name="odowheel_1">
@@ -99,15 +81,8 @@
       </material>
     </visual>
-    <collision>
-      <origin xyz="0 0 0" rpy="1.5707 0 0"/>
-      <geometry>
-        <cylinder radius="0.024" length="0.018"/>
-      </geometry>
-    </collision>
   </link>
   <link name="root"/>
   <joint name="fastened_2" type="fixed">
     <origin xyz="0 0 0" rpy="0 -0 3.14159"/>
-    <axis xyz="-0 -0 -1"/>
     <parent link="root"/>
     <child link="body"/>
@@ -124,63 +99,13 @@
     <child link="lidar"/>
   </joint>
-  <joint name="odowheel_x" type="continuous">
+  <joint name="odowheel_x" type="fixed">
     <origin xyz="-0.089012 -0.009 0.0286405" rpy="3.14159 -0 3.14159"/>
-    <axis xyz="0 -1 0"/>
     <parent link="body"/>
     <child link="odowheel"/>
   </joint>
-  <joint name="odowheel_y" type="continuous">
+  <joint name="odowheel_y" type="fixed">
     <origin xyz="0.014 -0.089012 0.0286405" rpy="0 0 -1.5708"/>
-    <axis xyz="0 -1 0"/>
     <parent link="body"/>
     <child link="odowheel_1"/>
   </joint>
-  <gazebo reference="lidar">
-    <sensor name="lidar" type="gpu_lidar">
-      <always_on>true</always_on>
-      <visualize>true</visualize>
-      <update_rate>10</update_rate>
-      <topic>scan</topic>
-      <gz_frame_id>lidar</gz_frame_id>
-      <lidar>
-        <scan>
-          <horizontal>
-            <samples>360</samples>
-            <resolution>1.000000</resolution>
-            <min_angle>0.000000</min_angle>
-            <max_angle>6.280000</max_angle>
-          </horizontal>
-        </scan>
-        <range>
-          <min>0.120000</min>
-          <max>3.5</max>
-          <resolution>0.015000</resolution>
-        </range>
-        <noise>
-          <type>gaussian</type>
-          <mean>0.0</mean>
-          <stddev>0.01</stddev>
-        </noise>
-      </lidar>
-    </sensor>
-  </gazebo>
-  <gazebo>
-    <plugin filename="ignition-gazebo-odometry-publisher-system" name="ignition::gazebo::systems::OdometryPublisher">
-      <odom_frame>odom</odom_frame>
-      <robot_base_frame>root</robot_base_frame>
-      <publish_odom_tf>true</publish_odom_tf>
-      <dimensions>3</dimensions>
-      <ros>
-        <argument>-p use_sim_time:=true</argument>
-      </ros>
-    </plugin>
-    <plugin filename="ignition-gazebo-joint-state-publisher-system" name="ignition::gazebo::systems::JointStatePublisher">
-      <joint_name>headlink</joint_name>
-      <joint_name>odowheel_x</joint_name>
-      <joint_name>odowheel_y</joint_name>
-      <ros>
-        <argument>-p use_sim_time:=true</argument>
-      </ros>
-    </plugin>
-  </gazebo>
 </robot>

Commit message: Add head pitch joint and RealSense camera mount to URDF
Adds a head_pitch link/joint (independent of the existing yaw-only
headlink) and a camera link fastened to it, so the head can carry a
tilting RealSense-style camera. Placeholder box geometry/mount origin
until a real mesh and measured offset exist; the sim package's copy of
this xacro wires up the matching gz sensor and controllers.

File: urdf/sentry.urdf.xacro (robot description, xacro)
@@ -47,4 +47,32 @@
       <material name="0.615686_0.811765_0.929412_0.000000_0.000000">
         <color rgba="0.615686 0.811765 0.929412 1"/>
+      </material>
+    </visual>
+  </link>
+  <!-- Pitch stage for the head, so a camera mounted on it can tilt
+       independently of the yaw-only headlink joint below. No mesh of its
+       own, just a bare kinematic link the camera is fastened to. -->
+  <link name="head_pitch">
+    <inertial>
+      <mass value="0.005"/>
+      <origin xyz="0 0 0" rpy="0 0 0"/>
+      <inertia ixx="1e-06" ixy="0" ixz="0" iyy="1e-06" iyz="0" izz="1e-06"/>
+    </inertial>
+  </link>
+  <!-- Approximates a RealSense D435 (90x25x25mm, 72g); no mesh exists for
+       it yet so a plain box visual stands in until one is added. -->
+  <link name="camera">
+    <inertial>
+      <mass value="0.072"/>
+      <origin xyz="0 0 0" rpy="0 0 0"/>
+      <inertia ixx="1.05e-05" ixy="0" ixz="0" iyy="5.4e-05" iyz="0" izz="5.4e-05"/>
+    </inertial>
+    <visual>
+      <origin xyz="0 0 0" rpy="0 0 0"/>
+      <geometry>
+        <box size="0.025 0.09 0.025"/>
+      </geometry>
+      <material name="0.1_0.1_0.1_0.000000_0.000000">
+        <color rgba="0.1 0.1 0.1 1"/>
       </material>
     </visual>
@@ -99,4 +127,19 @@
     <child link="lidar"/>
   </joint>
+  <!-- Pitch axis for the head-mounted camera. Placeholder mount point
+       (front-center of head, y-axis tilt) until it's positioned against
+       the real head mesh's geometry. -->
+  <joint name="headpitch" type="revolute">
+    <origin xyz="0.1 0 0" rpy="0 0 0"/>
+    <axis xyz="0 1 0"/>
+    <parent link="head"/>
+    <child link="head_pitch"/>
+    <limit lower="-0.6" upper="0.6" effort="5" velocity="3"/>
+  </joint>
+  <joint name="cameralink" type="fixed">
+    <origin xyz="0 0 0" rpy="0 0 0"/>
+    <parent link="head_pitch"/>
+    <child link="camera"/>
+  </joint>
   <joint name="odowheel_x" type="fixed">
     <origin xyz="-0.089012 -0.009 0.0286405" rpy="3.14159 -0 3.14159"/>

Commit message: Reposition headpitch mount above the lidar instead of head-front placeholder
Matches lidarlink's x/y origin on the head, raised ~5cm in z to clear it,
per user feedback that the pitch stage should sit on the existing head
structure near the lidar rather than an arbitrary front-center point.

File: urdf/sentry.urdf.xacro (robot description, xacro)
@@ -127,9 +127,9 @@
     <child link="lidar"/>
   </joint>
-  <!-- Pitch axis for the head-mounted camera. Placeholder mount point
-       (front-center of head, y-axis tilt) until it's positioned against
-       the real head mesh's geometry. -->
+  <!-- Pitch axis for the head-mounted camera. Mounted directly above the
+       lidar (same x/y as lidarlink's origin above, z raised ~5cm to clear
+       it) so the camera looks out from the same face of the head. -->
   <joint name="headpitch" type="revolute">
-    <origin xyz="0.1 0 0" rpy="0 0 0"/>
+    <origin xyz="-0.170562 -0.139254 0.1218" rpy="0 0 0"/>
     <axis xyz="0 1 0"/>
     <parent link="head"/>

Commit message: Center headpitch mount on the head (x/y=0), keep lidar-matched height
Per feedback: x/y should be centered on the head rather than offset to
match the lidar's mount point; only the z height (clearing the lidar)
was correct.

File: urdf/sentry.urdf.xacro (robot description, xacro)
@@ -127,9 +127,8 @@
     <child link="lidar"/>
   </joint>
-  <!-- Pitch axis for the head-mounted camera. Mounted directly above the
-       lidar (same x/y as lidarlink's origin above, z raised ~5cm to clear
-       it) so the camera looks out from the same face of the head. -->
+  <!-- Pitch axis for the head-mounted camera. Centered on the head (x/y=0)
+       at the same height as the lidar's mount z, raised ~5cm to clear it. -->
   <joint name="headpitch" type="revolute">
-    <origin xyz="-0.170562 -0.139254 0.1218" rpy="0 0 0"/>
+    <origin xyz="0 0 0.1218" rpy="0 0 0"/>
     <axis xyz="0 1 0"/>
     <parent link="head"/>

Commit message: Move camera forward on the head (+8cm x)
Per feedback: camera was centered inside the head; shift it forward so
it sits out past the head's front face.

File: urdf/sentry.urdf.xacro (robot description, xacro)
@@ -127,8 +127,10 @@
     <child link="lidar"/>
   </joint>
-  <!-- Pitch axis for the head-mounted camera. Centered on the head (x/y=0)
-       at the same height as the lidar's mount z, raised ~5cm to clear it. -->
+  <!-- Pitch axis for the head-mounted camera. Centered laterally (y=0) at
+       the same height as the lidar's mount z (raised ~5cm to clear it),
+       moved forward (+x) from head center so it sits out past the head's
+       front face rather than buried inside it. -->
   <joint name="headpitch" type="revolute">
-    <origin xyz="0 0 0.1218" rpy="0 0 0"/>
+    <origin xyz="0.08 0 0.1218" rpy="0 0 0"/>
     <axis xyz="0 1 0"/>
     <parent link="head"/>

Commit message: Counter-rotate camera mount to align with head mesh's visual rotation
The camera sat skewed relative to the rendered head because
headpitch's origin used rpy=0 (the link's raw frame) while head's own
<visual> block is rotated rpy="0 0 1.18195". Countering that rotation
on the mount aligns the camera box with the head as actually rendered.

File: urdf/sentry.urdf.xacro (robot description, xacro)
@@ -130,7 +130,10 @@
        the same height as the lidar's mount z (raised ~5cm to clear it),
        moved forward (+x) from head center so it sits out past the head's
-       front face rather than buried inside it. -->
+       front face rather than buried inside it. rpy counters head's own
+       <visual> mesh rotation (rpy="0 0 1.18195") so the camera box sits
+       flush/aligned with the head mesh as rendered instead of skewed
+       relative to it. -->
   <joint name="headpitch" type="revolute">
-    <origin xyz="0.08 0 0.1218" rpy="0 0 0"/>
+    <origin xyz="0.08 0 0.1218" rpy="0 0 -1.18195"/>
     <axis xyz="0 1 0"/>
     <parent link="head"/>

Commit message: Flip camera mount rotation sign (+1.18195 instead of -1.18195)
Previous sign was the wrong direction per feedback.

File: urdf/sentry.urdf.xacro (robot description, xacro)
@@ -130,10 +130,10 @@
        the same height as the lidar's mount z (raised ~5cm to clear it),
        moved forward (+x) from head center so it sits out past the head's
-       front face rather than buried inside it. rpy counters head's own
+       front face rather than buried inside it. rpy matches head's own
        <visual> mesh rotation (rpy="0 0 1.18195") so the camera box sits
        flush/aligned with the head mesh as rendered instead of skewed
        relative to it. -->
   <joint name="headpitch" type="revolute">
-    <origin xyz="0.08 0 0.1218" rpy="0 0 -1.18195"/>
+    <origin xyz="0.08 0 0.1218" rpy="0 0 1.18195"/>
     <axis xyz="0 1 0"/>
     <parent link="head"/>

Commit message: Try rpy z = 1.18195 - pi/2 for camera mount (still tuning)
Previous value (1.18195) was reported exactly 90deg off; trying the
smaller candidate first per feedback, to be confirmed against the live
camera feed once rviz is up.

File: urdf/sentry.urdf.xacro (robot description, xacro)
@@ -130,10 +130,11 @@
        the same height as the lidar's mount z (raised ~5cm to clear it),
        moved forward (+x) from head center so it sits out past the head's
-       front face rather than buried inside it. rpy matches head's own
-       <visual> mesh rotation (rpy="0 0 1.18195") so the camera box sits
-       flush/aligned with the head mesh as rendered instead of skewed
-       relative to it. -->
+       front face rather than buried inside it. rpy z tuned empirically
+       against the rendered scene/camera feed (head's own <visual> mesh
+       rotation is rpy="0 0 1.18195" but that alone overshot by 90deg;
+       this is that value minus pi/2, still being verified against the
+       live feed -- may need further tuning). -->
   <joint name="headpitch" type="revolute">
-    <origin xyz="0.08 0 0.1218" rpy="0 0 1.18195"/>
+    <origin xyz="0.08 0 0.1218" rpy="0 0 -0.38885"/>
     <axis xyz="0 1 0"/>
     <parent link="head"/>

Commit message: Confirm camera mount rotation correct; update comment

File: urdf/sentry.urdf.xacro (robot description, xacro)
@@ -131,8 +131,8 @@
        moved forward (+x) from head center so it sits out past the head's
        front face rather than buried inside it. rpy z tuned empirically
-       against the rendered scene/camera feed (head's own <visual> mesh
-       rotation is rpy="0 0 1.18195" but that alone overshot by 90deg;
-       this is that value minus pi/2, still being verified against the
-       live feed, may need further tuning). -->
+       against the rendered scene/camera feed and confirmed correct
+       (head's own <visual> mesh rotation is rpy="0 0 1.18195", but
+       matching that alone overshot by 90deg; this is that value minus
+       pi/2). -->
   <joint name="headpitch" type="revolute">
     <origin xyz="0.08 0 0.1218" rpy="0 0 -0.38885"/>

Commit message: Rotate camera 180 degrees (lens was facing backwards)

File: urdf/sentry.urdf.xacro (robot description, xacro)
@@ -131,10 +131,10 @@
        moved forward (+x) from head center so it sits out past the head's
        front face rather than buried inside it. rpy z tuned empirically
-       against the rendered scene/camera feed and confirmed correct
-       (head's own <visual> mesh rotation is rpy="0 0 1.18195", but
-       matching that alone overshot by 90deg; this is that value minus
-       pi/2). -->
+       against the rendered scene/camera feed (head's own <visual> mesh
+       rotation is rpy="0 0 1.18195"; this is that value minus pi/2, then
+       rotated a further 180deg per feedback that the lens was facing
+       backwards). -->
   <joint name="headpitch" type="revolute">
-    <origin xyz="0.08 0 0.1218" rpy="0 0 -0.38885"/>
+    <origin xyz="0.08 0 0.1218" rpy="0 0 2.75274"/>
     <axis xyz="0 1 0"/>
     <parent link="head"/>

Commit message: Rotate camera another 180 degrees (back to pre-flip value)

File: urdf/sentry.urdf.xacro (robot description, xacro)
@@ -132,9 +132,9 @@
        front face rather than buried inside it. rpy z tuned empirically
        against the rendered scene/camera feed (head's own <visual> mesh
-       rotation is rpy="0 0 1.18195"; this is that value minus pi/2, then
-       rotated a further 180deg per feedback that the lens was facing
-       backwards). -->
+       rotation is rpy="0 0 1.18195"; this is that value minus pi/2. A
+       subsequent 180deg flip turned out to be wrong too, so this is
+       back to that original value). -->
   <joint name="headpitch" type="revolute">
-    <origin xyz="0.08 0 0.1218" rpy="0 0 2.75274"/>
+    <origin xyz="0.08 0 0.1218" rpy="0 0 -0.38885"/>
     <axis xyz="0 1 0"/>
     <parent link="head"/>

Commit message: Move camera further forward (0.08m -> 0.16m)

File: urdf/sentry.urdf.xacro (robot description, xacro)
@@ -136,5 +136,5 @@
        back to that original value). -->
   <joint name="headpitch" type="revolute">
-    <origin xyz="0.08 0 0.1218" rpy="0 0 -0.38885"/>
+    <origin xyz="0.16 0 0.1218" rpy="0 0 -0.38885"/>
     <axis xyz="0 1 0"/>
     <parent link="head"/>

Commit message: Pull camera back a bit (0.16m -> 0.1m forward offset)

File: urdf/sentry.urdf.xacro (robot description, xacro)
@@ -136,5 +136,5 @@
        back to that original value). -->
   <joint name="headpitch" type="revolute">
-    <origin xyz="0.16 0 0.1218" rpy="0 0 -0.38885"/>
+    <origin xyz="0.1 0 0.1218" rpy="0 0 -0.38885"/>
     <axis xyz="0 1 0"/>
     <parent link="head"/>

Commit message: fix(description): adopt the team's low-resolution sentry CAD
Rebase CAD yaw -y onto head +x and exported 20-degree elevation onto
horizontal pitch zero. Import the IR apex, front bore muzzle, armor faces,
head heights and low-resolution visuals while retaining heading-fixed root.
Use the CAD lidar FOV reference (-0.105, -0.193326, 0.101293) in head with
scan-zero yaw -0.149533673 rad; retune the self-filter to 0.32-1.62 rad.

CAD archive SHA256:
0841b0ca27e54125ad8d962edf78dad97ce76198bb9d3b7c69036974ba32adff
The old-to-CAD XY change is 16.621 mm; CAD-to-Oct25 fit is 105.996 mm.
FOV zero/plane and the uneven-wheel clearance datum need hardware checks.

Validation: thornbots_pkg registered tests pass; xacro/check_urdf pass;
quality checker and actionlint pass. Coordinated sim integration records
baseline/changed regressions and outstanding armor/aiming assumptions.

File: urdf/sentry.urdf.xacro (robot description, xacro)
@@ -7,5 +7,5 @@
      under it on chassis_yaw, and the head hangs off root with headlink at
      the MCB's world head yaw, so lidar and camera never see chassis yaw.
-     The yaw bearing sits 0.2 mm off root's z axis; that offset is ignored. -->
+     The yaw bearing is centred on root; see README.md#robot-geometry. -->
 <robot name="sentry">
   <link name="root">
@@ -35,5 +35,5 @@
     <parent link="root"/>
     <child link="head"/>
-    <origin xyz="-0.000171242 9.52126e-05 0.248293" rpy="0 0 0"/>
+    <origin xyz="0 0 0.267503694" rpy="0 0 0"/>
     <axis xyz="0 0 1"/>
   </joint>
@@ -49,5 +49,5 @@
     <parent link="head"/>
     <child link="head_pitch"/>
-    <origin xyz="-0.00760542 -0.100122 0.14235" rpy="0 0 0"/>
+    <origin xyz="0 0 0.136" rpy="0 0 0"/>
     <axis xyz="0 1 0"/>
     <limit lower="-0.6" upper="0.6" effort="200" velocity="10"/>
@@ -170,5 +170,5 @@
     <parent link="body"/>
     <child link="armor_0"/>
-    <origin xyz="0.178162 0.178426 0.230361" rpy="0 -0.261856 0.785329"/>
+    <origin xyz="0.204139959 0.150682952 0.148603392" rpy="0 -0.261799339 0.635864487"/>
   </joint>
   <link name="armor_1">
@@ -181,5 +181,5 @@
     <parent link="body"/>
     <child link="armor_1"/>
-    <origin xyz="-0.177935 0.177863 0.135661" rpy="0 -0.261856 2.35613"/>
+    <origin xyz="-0.148299431 0.200910863 0.25248797" rpy="0 -0.261797504 2.206660314"/>
   </joint>
   <link name="armor_2">
@@ -192,5 +192,5 @@
     <parent link="body"/>
     <child link="armor_2"/>
-    <origin xyz="-0.178505 -0.178235 0.230361" rpy="0 -0.261856 -2.35627"/>
+    <origin xyz="-0.204139942 -0.150683009 0.148603318" rpy="0 -0.261796504 -2.505724829"/>
   </joint>
   <link name="armor_3">
@@ -203,5 +203,5 @@
     <parent link="body"/>
     <child link="armor_3"/>
-    <origin xyz="0.177593 -0.177673 0.135661" rpy="0 -0.261856 -0.785464"/>
+    <origin xyz="0.148299403 -0.200910883 0.252487973" rpy="0 -0.261799535 -0.934934345"/>
   </joint>
   <link name="lidar"/>
@@ -209,5 +209,5 @@
     <parent link="head"/>
     <child link="lidar"/>
-    <origin xyz="-0.119391 -0.18501 0.0968001" rpy="0 0 0"/>
+    <origin xyz="-0.105 -0.193326 0.101293" rpy="0 0 -0.149533673"/>
   </joint>
   <link name="camera"/>
@@ -215,8 +215,8 @@
     <parent link="head_pitch"/>
     <child link="camera"/>
-    <origin xyz="0.0920381 0.0948673 0.0566588" rpy="0 0 0"/>
-  </joint>
-  <!-- Where the shot leaves: on the pitch axis, between the flywheels
-       (sentry_v2 CAD), pointing along head_pitch +x. Not in the generated
+    <origin xyz="0.095699877 -0.011500052 0.055000043" rpy="0 0 0"/>
+  </joint>
+  <!-- Where the shot leaves: at the front bore centre of the 2026-10-26 CAD,
+       pointing along head_pitch +x. Not in the generated
        model; sim/urdf/sentry_v2.urdf.xacro adds the same frame. -->
   <link name="muzzle"/>
@@ -224,5 +224,5 @@
     <parent link="head_pitch"/>
     <child link="muzzle"/>
-    <origin xyz="0 0.1128 0" rpy="0 0 0"/>
+    <origin xyz="0.1729764 0.00190269 0" rpy="0 0 0"/>
   </joint>
 </robot>

Commit message: fix(description): preserve the muzzle pitch-axis contract
Keep the CAD lateral offset while restoring the pitch-invariant aiming origin between the flywheels. The bore-front location is documented separately.

File: urdf/sentry.urdf.xacro (robot description, xacro)
@@ -217,12 +217,12 @@
     <origin xyz="0.095699877 -0.011500052 0.055000043" rpy="0 0 0"/>
   </joint>
-  <!-- Where the shot leaves: at the front bore centre of the 2026-10-26 CAD,
-       pointing along head_pitch +x. Not in the generated
-       model; sim/urdf/sentry_v2.urdf.xacro adds the same frame. -->
+  <!-- Aiming origin on the pitch axis, between the flywheels, pointing
+       along head_pitch +x. Only the lateral offset comes from the CAD;
+       sim/urdf/sentry_v2.urdf.xacro adds the same frame. -->
   <link name="muzzle"/>
   <joint name="muzzlelink" type="fixed">
     <parent link="head_pitch"/>
     <child link="muzzle"/>
-    <origin xyz="0.1729764 0.00190269 0" rpy="0 0 0"/>
+    <origin xyz="0 0.00190269 0" rpy="0 0 0"/>
   </joint>
 </robot>

Commit message: feat: expose lidar mount and blind sector launch arguments
Pass lidar_x/y/z/yaw into xacro and scan-frame blind bounds into the
self-filter. Normalize sector bounds to support the provisional yaw A/B
sector crossing scan zero; keep the default mount and masking unchanged.

Validation: nightly 2290338 and default xacro outputs have an empty diff
and SHA-256 201a0f0a2e783943fa4968c9209b1aa54da117952599d240e73ff4acde207e36.
Package tests: 140 passed. Host Python 3.12 quality and actionlint pass.
Isolated auto.launch.py dry run confirms head->lidar CAD xyz
(-0.105, -0.193326, 0.101293), yaw 0.597, and forwarded blind bounds.
Synthetic scans verify all 720 default bins against the former algorithm,
signed/wrapped sectors and inclusive endpoints. No physical robot runs.

File: urdf/sentry.urdf.xacro (robot description, xacro)
@@ -8,5 +8,10 @@
      the MCB's world head yaw, so lidar and camera never see chassis yaw.
      The yaw bearing sits 0.2 mm off root's z axis; that offset is ignored. -->
-<robot name="sentry">
+<robot name="sentry" xmlns:xacro="http://www.ros.org/wiki/xacro">
+  <xacro:arg name="lidar_x" default="-0.119391"/>
+  <xacro:arg name="lidar_y" default="-0.18501"/>
+  <xacro:arg name="lidar_z" default="0.0968001"/>
+  <xacro:arg name="lidar_yaw" default="0"/>
+  <xacro:property name="lidar_yaw" value="$(arg lidar_yaw)"/>
   <link name="root">
     <visual>
@@ -209,5 +214,5 @@
     <parent link="head"/>
     <child link="lidar"/>
-    <origin xyz="-0.119391 -0.18501 0.0968001" rpy="0 0 0"/>
+    <origin xyz="$(arg lidar_x) $(arg lidar_y) $(arg lidar_z)" rpy="0 0 ${lidar_yaw}"/>
   </joint>
   <link name="camera"/>
