Commit message: fix(lidar): use the Oct 26 measured mount and self-filter
Use CAD head-frame xyz (-0.105, -0.193326, 0.101293), five-pose joint-fit scan-zero yaw 0.5907 rad, and robot-verified scan-frame sector -0.5585..1.0123 rad. Evidence: ~/ros2_ws/robot-session-20261026/evidence-1/{headturn-yaw-joint,1a-level-probe,1c-old-shift,1d-new-shift}.txt on the Mac mini; workspace docs/investigations/lidar-mount-2026-10-26.md records provenance. Supersedes the authored CAD FOV-marker yaw.

Validation: isolated Jazzy agent container, colcon test thornbots_pkg: 142 tests, zero errors/failures/skips. Host Python 3.12 quality and actionlint pass. No robot run.

File: urdf/sentry.urdf.xacro (robot description, xacro)
@@ -9,9 +9,8 @@
      The yaw bearing sits 0.2 mm off root's z axis; that offset is ignored. -->
 <robot name="sentry" xmlns:xacro="http://www.ros.org/wiki/xacro">
-  <xacro:arg name="lidar_x" default="-0.119391"/>
-  <xacro:arg name="lidar_y" default="-0.18501"/>
-  <xacro:arg name="lidar_z" default="0.0968001"/>
-  <xacro:arg name="lidar_yaw" default="0"/>
-  <xacro:property name="lidar_yaw" value="$(arg lidar_yaw)"/>
+  <xacro:arg name="lidar_x" default="-0.105"/>
+  <xacro:arg name="lidar_y" default="-0.193326"/>
+  <xacro:arg name="lidar_z" default="0.101293"/>
+  <xacro:arg name="lidar_yaw" default="0.5907"/>
   <link name="root">
     <visual>
@@ -214,5 +213,5 @@
     <parent link="head"/>
     <child link="lidar"/>
-    <origin xyz="$(arg lidar_x) $(arg lidar_y) $(arg lidar_z)" rpy="0 0 ${lidar_yaw}"/>
+    <origin xyz="$(arg lidar_x) $(arg lidar_y) $(arg lidar_z)" rpy="0 0 $(arg lidar_yaw)"/>
   </joint>
   <link name="camera"/>

Commit message: fix(urdf): put the camera frame on the D435's RGB lens
/cv/panel_detections are deprojected with the colour intrinsics, so the
camera frame must be the RGB lens: 32.5 mm to the camera's left of the
CAD cover centre (17.5 mm to the depth origin + 15 mm to colour; MCBV3's
cameraXoffset -0.0325 records the same). At the cover centre every aim
point landed 32.5 mm right of its panel on the real robot.

Matches sim/urdf/sentry_v2 (test_cv_bench checks). colcon test sim +
thornbots_pkg 432/432; aiming bench 10/10; estimation bench 12/12.

File: urdf/sentry.urdf.xacro (robot description, xacro)
@@ -215,9 +215,12 @@
     <origin xyz="$(arg lidar_x) $(arg lidar_y) $(arg lidar_z)" rpy="0 0 $(arg lidar_yaw)"/>
   </joint>
+  <!-- The D435's RGB lens, which /cv/panel_detections are deprojected from:
+       the CAD camera cover's centre plus 32.5 mm to the camera's left
+       (sim/urdf/sentry_v2.yaml sensor_offsets). -->
   <link name="camera"/>
   <joint name="cameralink" type="fixed">
     <parent link="head_pitch"/>
     <child link="camera"/>
-    <origin xyz="0.0920381 0.0948673 0.0566588" rpy="0 0 0"/>
+    <origin xyz="0.0920381 0.127367 0.0566588" rpy="0 0 0"/>
   </joint>
   <!-- Where the shot leaves: on the pitch axis, between the flywheels
